File: obc_board/cubesat_obc.kicad_pcb (KiCad board)
At the start: 2 copper layers, 96 x 89.9 mm, 156 parts, among them J1 Conn_01x04_Female, J10 FSI-110-03-X-D-AD-SD-K-TR, J11 FSI-110-03-X-D-AD-SD-K-TR, J2 Conn_01x04_Female, J3 Conn_ARM_JTAG_SWD_20, J4 Micro_SD_Card, J5 Conn_01x02_Female, J6 Conn_01x02_Female, J7 Conn_01x02_Female, J8 Conn_01x02_Female, J9 SAMTEC-MMS-110-01-X-DV, U1 PC104, U10 BMI160, U11 BMM150, U12 LTC4304CMSTRPBF, U13 LTC4304CMSTRPBF, U2 AT45DB041E-SSHN-B, U3 AT45DB041E-SSHN-B, U4 STM32L552ZE, U5 LTC4304CMSTRPBF, U6 MCP9600-E_MX, U7 MCP9600-E_MX, U8 MCP9600-E_MX, U9 MCP9600-E_MX

Commit message: pcb layout
Parts:
- removed the C34 at (156.0, 140.7)
- removed the FL1 at (128.1, 156.4)
- removed the J9 at (128.6, 137.5)
- removed the R12 at (76.0, 160.0)
- removed the R13 at (93.7, 139.7)
- removed the R14 at (69.1, 164.6)
- removed the U1 at (45.2, 117.1)
- added C36: 100n, Capacitor_SMD:C_0402_1005Metric, F.Cu at (153.2, 101.5)
- added C37: 100n, Capacitor_SMD:C_0402_1005Metric, F.Cu at (153.2, 90.9)
- added C38: 100n, Capacitor_SMD:C_0402_1005Metric, F.Cu at (162.3, 106.3)
- added C39: 100n, Capacitor_SMD:C_0402_1005Metric, F.Cu at (163.8, 126.7)
- added H1: MountingHole, MountingHole:MountingHole_3.2mm_M3_DIN965_Pad, F.Cu at (110.7, 55.8)
- added H10: MountingHole, Mounting_Wuerth:Mounting_Wuerth_WA-SMSI-M3_H3mm_9774030360, F.Cu at (186.5, 132.0)
- added H11: MountingHole, Mounting_Wuerth:Mounting_Wuerth_WA-SMSI-M3_H3mm_9774030360, F.Cu at (186.5, 98.3)
- added H12: MountingHole, Mounting_Wuerth:Mounting_Wuerth_WA-SMSI-M3_H3mm_9774030360, F.Cu at (186.5, 88.3)
- added H2: MountingHole, MountingHole:MountingHole_3.2mm_M3_DIN965_Pad, F.Cu at (196.5, 133.3)
- added H3: MountingHole, MountingHole:MountingHole_3.2mm_M3_DIN965_Pad, F.Cu at (196.5, 53.3)
- added H4: MountingHole, MountingHole:MountingHole_3.2mm_M3_DIN965_Pad, F.Cu at (110.7, 129.5)
- added H5: MountingHole, Mounting_Wuerth:Mounting_Wuerth_WA-SMSI-M3_H3mm_9774030360, F.Cu at (127.7, 88.3)
- added H6: MountingHole, Mounting_Wuerth:Mounting_Wuerth_WA-SMSI-M3_H3mm_9774030360, F.Cu at (127.7, 98.3)
- added H7: MountingHole, Mounting_Wuerth:Mounting_Wuerth_WA-SMSI-M3_H3mm_9774030360, F.Cu at (127.7, 54.5)
- added H8: MountingHole, Mounting_Wuerth:Mounting_Wuerth_WA-SMSI-M3_H3mm_9774030360, F.Cu at (186.5, 54.5)
- added H9: MountingHole, Mounting_Wuerth:Mounting_Wuerth_WA-SMSI-M3_H3mm_9774030360, F.Cu at (127.7, 132.0)
- added J1: Conn_01x04_Female, Connector_Molex:Molex_PicoBlade_53261-0471_1x04-1MP_P1.25mm_Horizontal, B.Cu at (137.8, 51.7)
- added J2: Conn_01x04_Female, Connector_Molex:Molex_PicoBlade_53261-0471_1x04-1MP_P1.25mm_Horizontal, B.Cu at (150.6, 51.9)
- added J4: Conn_01x04_Female, Connector_Molex:Molex_PicoBlade_53261-0471_1x04-1MP_P1.25mm_Horizontal, B.Cu at (176.3, 51.9)
- added J5: Conn_01x05_Female, Connector_Molex:Molex_PicoBlade_53261-0571_1x05-1MP_P1.25mm_Horizontal, F.Cu at (196.7, 64.4)
- added J8: Conn_01x08_Female, Connector_Molex:Molex_PicoBlade_53261-0871_1x08-1MP_P1.25mm_Horizontal, B.Cu at (196.4, 72.1)
- added R51: 0, Resistor_SMD:R_0402_1005Metric, F.Cu at (178.9, 115.8)
- added R52: 0, Resistor_SMD:R_0402_1005Metric, F.Cu at (178.9, 110.9)
- added R54: 0, Resistor_SMD:R_0402_1005Metric, F.Cu at (179.0, 114.2)
- added R56: 0, Resistor_SMD:R_0402_1005Metric, F.Cu at (179.0, 112.6)
- added R71: 0, Resistor_SMD:R_0402_1005Metric, F.Cu at (134.6, 85.6)
- added R72: 0, Resistor_SMD:R_0402_1005Metric, F.Cu at (134.6, 93.2)
- added R73: 0, Resistor_SMD:R_0402_1005Metric, F.Cu at (135.8, 85.5)
- added R74: 0, Resistor_SMD:R_0402_1005Metric, F.Cu at (135.9, 93.2)
- added R75: 0, Resistor_SMD:R_0402_1005Metric, F.Cu at (137.1, 85.5)
- added R76: 0, Resistor_SMD:R_0402_1005Metric, F.Cu at (137.2, 93.2)
- added R77: 0, Resistor_SMD:R_0402_1005Metric, F.Cu at (138.4, 85.5)
- added R78: 0, Resistor_SMD:R_0402_1005Metric, F.Cu at (138.4, 93.2)
- added R79: 0, Resistor_SMD:R_0402_1005Metric, F.Cu at (139.6, 85.5)
- added R80: 0, Resistor_SMD:R_0402_1005Metric, F.Cu at (139.7, 93.3)
- added R81: 0, Resistor_SMD:R_0402_1005Metric, F.Cu at (140.9, 85.5)
- added R82: 0, Resistor_SMD:R_0402_1005Metric, F.Cu at (140.9, 93.3)
- added R83: 0, Resistor_SMD:R_0402_1005Metric, F.Cu at (134.6, 89.3)
- added R84: 0, Resistor_SMD:R_0402_1005Metric, F.Cu at (134.6, 97.7)
- added R85: 0, Resistor_SMD:R_0402_1005Metric, F.Cu at (135.8, 89.3)
- added R86: 0, Resistor_SMD:R_0402_1005Metric, F.Cu at (135.8, 97.7)
- added R87: 0, Resistor_SMD:R_0402_1005Metric, F.Cu at (137.1, 89.3)
- added R88: 0, Resistor_SMD:R_0402_1005Metric, F.Cu at (137.1, 97.7)
- added R89: 0, Resistor_SMD:R_0402_1005Metric, F.Cu at (138.4, 89.3)
- added R90: 0, Resistor_SMD:R_0402_1005Metric, F.Cu at (138.4, 97.7)
- added R91: 0, Resistor_SMD:R_0402_1005Metric, F.Cu at (139.6, 89.4)
- added R92: 0, Resistor_SMD:R_0402_1005Metric, F.Cu at (139.6, 97.7)
- added R93: 0, Resistor_SMD:R_0402_1005Metric, F.Cu at (140.9, 89.4)
- added R94: 0, Resistor_SMD:R_0402_1005Metric, F.Cu at (140.9, 97.7)
- added R95: 10k, Resistor_SMD:R_0402_1005Metric, B.Cu at (140.5, 106.2)
- added R96: 10k, Resistor_SMD:R_0402_1005Metric, B.Cu at (142.5, 106.2)
- added R97: 10k, Resistor_SMD:R_0402_1005Metric, B.Cu at (145.4, 88.1)
- added R98: 10k, Resistor_SMD:R_0402_1005Metric, B.Cu at (147.7, 88.1)
- added U13: PC104, cubesat_obc:PC104-Standard, F.Cu at (110.6, 129.4)
- C1, C16, C2, C23, C26, C27, C28, C29, D1, D10, D11, D12, D13, D14, D15, D16, D2, D3, D4, D5, D6, D7, D8, D9, L1, L2, L3, L4, L5, L6, L7, L8: moved to B.Cu
- C18: footprint Capacitor_THT:CP_Radial_D5.0mm_P2.00mm -> Capacitor_SMD:CP_Elec_4x5.3; moved to B.Cu
- C19, C20, C25: footprint Capacitor_THT:CP_Radial_D5.0mm_P2.00mm -> Capacitor_SMD:CP_Elec_4x5.3
- C34: renamed from C35; footprint Capacitor_THT:CP_Radial_D5.0mm_P2.00mm -> Capacitor_SMD:CP_Elec_4x5.3
- C35: renamed from C36; footprint Capacitor_THT:CP_Radial_D5.0mm_P2.00mm -> Capacitor_SMD:CP_Elec_4x5.3
- FL1: renamed from FL2; moved to B.Cu
- FL2: renamed from FL3; moved to B.Cu
- J10: renamed from J5; footprint Connector_Molex:Molex_PicoBlade_53398-0271_1x02-1MP_P1.25mm_Vertical -> Connector_Molex:Molex_PicoBlade_53261-0271_1x02-1MP_P1.25mm_Horizontal; moved to B.Cu
- J11: renamed from J6; footprint Connector_Molex:Molex_PicoBlade_53398-0271_1x02-1MP_P1.25mm_Vertical -> Connector_Molex:Molex_PicoBlade_53261-0271_1x02-1MP_P1.25mm_Horizontal; moved to B.Cu
- J12: renamed from J7; footprint Connector_Molex:Molex_PicoBlade_53398-0271_1x02-1MP_P1.25mm_Vertical -> Connector_Molex:Molex_PicoBlade_53261-0271_1x02-1MP_P1.25mm_Horizontal; moved to B.Cu
- J13: renamed from J8; footprint Connector_Molex:Molex_PicoBlade_53398-0271_1x02-1MP_P1.25mm_Vertical -> Connector_Molex:Molex_PicoBlade_53261-0271_1x02-1MP_P1.25mm_Horizontal; moved to B.Cu
- J3: value Conn_ARM_JTAG_SWD_20 -> Conn_01x04_Female; footprint Connector_IDC:IDC-Header_2x10_P2.54mm_Vertical -> Connector_Molex:Molex_PicoBlade_53261-0471_1x04-1MP_P1.25mm_Horizontal; moved to B.Cu
- J6: renamed from J1; footprint Connector_Molex:Molex_PicoBlade_53398-0471_1x04-1MP_P1.25mm_Vertical -> Connector_Molex:Molex_PicoBlade_53261-0471_1x04-1MP_P1.25mm_Horizontal; moved to B.Cu
- J7: renamed from J2; footprint Connector_Molex:Molex_PicoBlade_53398-0471_1x04-1MP_P1.25mm_Vertical -> Connector_Molex:Molex_PicoBlade_53261-0471_1x04-1MP_P1.25mm_Horizontal; moved to B.Cu
- J9: renamed from J4; moved to B.Cu
- R22: renamed from R25; moved to B.Cu
- R23: renamed from R26; moved to B.Cu
- R24: renamed from R27; moved to B.Cu
- R25: renamed from R28; moved to B.Cu
- R26: renamed from R29; moved to B.Cu
- R27: renamed from R30; moved to B.Cu
- R28: renamed from R31; moved to B.Cu
- R29: renamed from R32; moved to B.Cu
- R30: renamed from R33; moved to B.Cu
- R31: renamed from R34; moved to B.Cu
- R37: renamed from R40; moved to B.Cu
- R38: renamed from R41; moved to B.Cu
- R39: renamed from R42; moved to B.Cu
- R40: renamed from R43; moved to B.Cu
- R41: renamed from R44; moved to B.Cu
- R42: renamed from R45; moved to B.Cu
- R43: renamed from R46; moved to B.Cu
- R44: renamed from R47; moved to B.Cu
- R45: renamed from R48; moved to B.Cu
- R46: renamed from R49; moved to B.Cu
- U1: renamed from U2; moved to B.Cu
- U2: renamed from U3; moved to B.Cu
- U3: renamed from U4; moved to B.Cu
- U4: renamed from U5; moved to B.Cu
- U5: renamed from U6; moved to B.Cu
- U6: renamed from U7; moved to B.Cu
- U7: renamed from U8; moved to B.Cu
- U8: renamed from U9; moved to B.Cu
- moved C19 155.2 mm to (195.6, 83.9)
- moved R14 154.8 mm to (173.1, 60.3)
- moved J9 154.6 mm to (146.4, 128.8)
- moved R20 152.6 mm to (173.1, 66.7)
- moved R13 147.7 mm to (169.5, 61.8)
- moved J3 147.1 mm to (163.4, 51.9)
- moved C15 144.7 mm to (144.4, 63.3), turned to 180 degrees
- moved C20 142.0 mm to (195.5, 93.3)
- moved R21 140.9 mm to (173.1, 68.3)
- moved C17 140.3 mm to (143.4, 65.7), turned to 90 degrees
- moved R19 139.5 mm to (169.5, 68.3)
- moved R17 139.2 mm to (176.7, 61.8)
- moved C22 135.6 mm to (164.9, 81.1), turned to 270 degrees
- moved C16 135.4 mm to (138.8, 74.9)
- moved C11 130.8 mm to (161.0, 74.4), turned to 270 degrees
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- renumbered J10 to J14, J11 to J15, R15 to R12, R16 to R13, R17 to R14, R18 to R15, R19 to R16, R20 to R17, R21 to R18, R22 to R19, R23 to R20, R24 to R21, R35 to R32, R36 to R33, R37 to R34, R38 to R35, R39 to R36, R50 to R47, R51 to R48, R52 to R49, R53 to R50, R54 to R53, R56 to R57, R57 to R58, R58 to R59, R59 to R60, R60 to R61, R61 to R62, R62 to R63, R63 to R64, R64 to R65, R65 to R66, R66 to R67, R67 to R68, R68 to R69, R69 to R70, U11 to U10, U12 to U11, U13 to U12, U10 to U9
Connections:
- net Net-(U4-Pad93) renamed /mcu/PG8
- C1 pad 1: /3V3_4 -> /3V3_3
- C11 pad 2: /3V3_4 -> /3V3_3
- C12 pad 2: /3V3_4 -> /3V3_3
- C13 pad 1: /3V3_4 -> /3V3_3
- C14 pad 1: /3V3_4 -> /3V3_3
- C15 pad 1: /3V3_4 -> /3V3_3
- C16 pad 2: /3V3_4 -> /3V3_3
- C17 pad 2: /3V3_4 -> /3V3_3
- C18 pad 1: /3V3_4 -> /3V3_3
- C19 pad 1: /3V3_4 -> /3V3_3
- C2 pad 1: /3V3_4 -> /3V3_3
- C20 pad 1: /3V3_4 -> /3V3_3
- C21 pad 2: /3V3_4 -> /3V3_3
- C22 pad 2: /3V3_4 -> /3V3_3
- C23 pad 2: /3V3_4 -> /3V3_3
- C24 pad 2: /3V3_4 -> /3V3_3
- C25 pad 1: /3V3_4 -> /3V3_3
- C3 pad 1: /3V3_4 -> /3V3_3
- C30 pad 1: /3V3_4 -> /3V3_3
- C31 pad 1: /3V3_4 -> /3V3_3
- C32 pad 1: /3V3_4 -> /3V3_3
- C33 pad 1: /3V3_4 -> /3V3_3
- C4 pad 1: /3V3_4 -> /3V3_3
- C5 pad 1: /3V3_4 -> /3V3_3
- C8 pad 1: /3V3_4 -> /3V3_3
- D11 pad 1: /3V3_4 -> /sensors/3V3_2
- D12 pad 1: /3V3_4 -> /sensors/3V3_4
- D13 pad 1: /3V3_4 -> /sensors/3V3_2
- D15 pad 1: /3V3_4 -> /sensors/3V3_4
- D3 pad 1: /3V3_4 -> /sensors/3V3_1
- D4 pad 1: /3V3_4 -> /sensors/3V3_3
- D5 pad 1: /3V3_4 -> /sensors/3V3_1
- D7 pad 1: /3V3_4 -> /sensors/3V3_3
- J3 pad 1: /3V3_4 -> /VCC
- J3 pad 2: /3V3_4 -> /TX3
- J3 pad 3: /mcu/NJRST -> /RX3
- J9 pad 4: /3V3_4 -> /3V3_3
- R10 pad 1: /3V3_4 -> /3V3_3
- R11 pad 1: /3V3_4 -> /3V3_3
- R12 pad 1: /3V3_4 -> /3V3_3
- R13 pad 1: /3V3_4 -> /3V3_3
- R14 pad 1: /3V3_4 -> /3V3_3
- R15 pad 1: /3V3_4 -> /3V3_3
- R16 pad 1: /3V3_4 -> /3V3_3
- R17 pad 1: /3V3_4 -> /3V3_3
- R18 pad 1: /SDA1 -> /SDA2
- R18 pad 2: /3V3_4 -> /3V3_3
- R19 pad 1: /SCL1 -> /SCL2
- R19 pad 2: /3V3_4 -> /3V3_3
- R20 pad 2: /3V3_4 -> /3V3_3
- R21 pad 2: /3V3_4 -> /3V3_3
- R26 pad 1: /3V3_4 -> /sensors/3V3_1
- R29 pad 1: /3V3_4 -> /sensors/3V3_3
- R3 pad 1: /3V3_4 -> /3V3_3
- R32 pad 1: /3V3_4 -> /sensors/3V3_3
- R34 pad 1: /3V3_4 -> /3V3_3
- R35 pad 1: /3V3_4 -> /3V3_3
- R36 pad 1: /3V3_4 -> /3V3_3
- R41 pad 1: /3V3_4 -> /sensors/3V3_2
- R44 pad 1: /3V3_4 -> /sensors/3V3_4
- R47 pad 1: /3V3_4 -> /sensors/3V3_2
- R49 pad 1: /3V3_4 -> /sensors/3V3_4
- R5 pad 1: /3V3_4 -> /3V3_3
- R53 pad 1: /3V3_4 -> /3V3_3
- R55 pad 1: /3V3_4 -> /3V3_3
- R6 pad 1: /3V3_4 -> /3V3_3
- R7 pad 1: /3V3_4 -> /3V3_3
- R8 pad 1: /3V3_4 -> /3V3_3
- R9 pad 1: /3V3_4 -> /3V3_3
- U1 pad 6: /3V3_4 -> /3V3_3
- U10 pad B2: /3V3_4 -> /3V3_3
- U10 pad E5: /3V3_4 -> /3V3_3
- U2 pad 6: /3V3_4 -> /3V3_3
- U3 pad 106: /3V3_4 -> /3V3_3
- U3 pad 108: /3V3_4 -> /3V3_3
- U3 pad 121: /3V3_4 -> /3V3_3
- U3 pad 131: /3V3_4 -> /3V3_3
- U3 pad 144: /3V3_4 -> /3V3_3
- U3 pad 17: /3V3_4 -> /3V3_3
- U3 pad 33: /3V3_4 -> /3V3_3
- U3 pad 39: /3V3_4 -> /3V3_3
- U3 pad 52: /3V3_4 -> /3V3_3
- U3 pad 6: Net-(U4-Pad6) (its old number) -> /3V3_P
- U3 pad 62: /3V3_4 -> /3V3_3
- U3 pad 72: /3V3_4 -> /3V3_3
- U3 pad 84: /3V3_4 -> /3V3_3
- U3 pad 91: Net-(U4-Pad91) -> /CS1
- U3 pad 92: Net-(U4-Pad92) -> /CS2
- U3 pad 95: /3V3_4 -> /3V3_3
- U4 pad 10: /3V3_4 -> /3V3_3
- U5 pad 8: /3V3_4 -> /sensors/3V3_1
- U6 pad 8: /3V3_4 -> /sensors/3V3_3
- U7 pad 8: /3V3_4 -> /sensors/3V3_2
- U8 pad 8: /3V3_4 -> /sensors/3V3_4
- U9 pad 5: /3V3_4 -> /3V3_3
- U9 pad 8: /3V3_4 -> /3V3_3
Other:
- board size 96 x 89.9 mm -> 92 x 88.9 mm

Commit message: layout
Parts:
- added C40: 100n, Capacitor_SMD:C_0402_1005Metric, F.Cu at (144.8, 115.6)
- added C41: 100n, Capacitor_SMD:C_0402_1005Metric, B.Cu at (144.8, 111.8)
- added C42: 100n, Capacitor_SMD:C_0402_1005Metric, F.Cu at (147.3, 108.7)
- added C43: 100n, Capacitor_SMD:C_0402_1005Metric, F.Cu at (144.8, 114.3)
- added R100: 10k, Resistor_SMD:R_0402_1005Metric, B.Cu at (138.4, 118.1)
- added R101: 10k, Resistor_SMD:R_0402_1005Metric, B.Cu at (139.7, 119.4)
- added R102: 10k, Resistor_SMD:R_0402_1005Metric, B.Cu at (142.7, 117.2)
- added R103: 100k, Resistor_SMD:R_0402_1005Metric, F.Cu at (135.9, 52.1)
- added R104: 100k, Resistor_SMD:R_0402_1005Metric, F.Cu at (148.6, 52.1)
- added R105: 100k, Resistor_SMD:R_0402_1005Metric, F.Cu at (161.3, 52.1)
- added R106: 100k, Resistor_SMD:R_0402_1005Metric, F.Cu at (174.0, 52.1)
- added R107: 100k, Resistor_SMD:R_0402_1005Metric, F.Cu at (135.9, 50.8)
- added R108: 100k, Resistor_SMD:R_0402_1005Metric, F.Cu at (148.6, 50.8)
- added R109: 100k, Resistor_SMD:R_0402_1005Metric, F.Cu at (161.3, 50.8)
- added R110: 100k, Resistor_SMD:R_0402_1005Metric, F.Cu at (174.0, 50.8)
- added R99: 10k, Resistor_SMD:R_0402_1005Metric, B.Cu at (138.4, 116.8)
- added U14: MAX14830, Package_DFN_QFN:TQFN-48-1EP_7x7mm_P0.5mm_EP5.1x5.1mm, B.Cu at (139.7, 111.8)
- added Y1: 32.768kHz, Crystal:Crystal_SMD_3215-2Pin_3.2x1.5mm, F.Cu at (146.1, 78.8)
- added Y2: 8MHz, Crystal:Crystal_SMD_3225-4Pin_3.2x2.5mm, B.Cu at (137.6, 69.7)
- added Y3: 4MHz, Crystal:Crystal_SMD_MicroCrystal_CC1V-T1A-2Pin_8.0x3.7mm, B.Cu at (151.1, 115.6)
- C10: moved to B.Cu
- moved C7 123.4 mm to (148.6, 80.0)
- moved C9 122.2 mm to (134.6, 69.8), turned to 180 degrees
- moved C6 116.6 mm to (148.6, 77.5)
- moved C10 89.6 mm to (138.4, 66.0)
- moved J4 0.60 mm to (175.8, 52.1)
- moved J3 0.43 mm to (163.1, 52.1)
- moved J1 0.36 mm to (137.7, 52.1)
- moved J2 0.32 mm to (150.4, 52.1)
Connections:
- J1 pad 2: /TX1 -> /uart_expander/TX0
- J1 pad 3: /RX1 -> /uart_expander/RX0
- J14 pad 17: /RX1 -> /TX1
- J14 pad 18: /RX2 -> /TX2
- J14 pad 19: /TX1 -> /RX1
- J14 pad 20: /TX2 -> /RX2
- J15 pad 17: /RX1 -> /TX3
- J15 pad 18: /RX2 -> /TX4
- J15 pad 19: /TX1 -> /RX3
- J15 pad 20: /TX2 -> /RX4
- J2 pad 2: /TX2 -> /uart_expander/TX1
- J2 pad 3: /RX2 -> /uart_expander/RX1
- J3 pad 2: /TX3 -> /uart_expander/TX2
- J3 pad 3: /RX3 -> /uart_expander/RX2
- J4 pad 2: /TX4 -> /uart_expander/TX3
- J4 pad 3: /RX4 -> /uart_expander/RX3
- J5 pad 4: Net-(J5-Pad4) -> /CS3
- R84 pad 1: /stacking_connector/3V3_4 -> /VCC
- R86 pad 1: /stacking_connector/3V3_4 -> /VCC
- R88 pad 1: /stacking_connector/3V3_4 -> /VCC
- R90 pad 1: /stacking_connector/3V3_4 -> /VCC
- R92 pad 1: /stacking_connector/3V3_4 -> /VCC
- R94 pad 1: /stacking_connector/3V3_4 -> /VCC
- U3 pad 19: /CS1 -> /INT
- U3 pad 20: /CS2 -> /RST
- U3 pad 90: Net-(U3-Pad90) -> /EXP
- U3 pad 93: /mcu/PG8 -> /CS3
Other:
- rule via_min_drill: 0.3 -> 0.2

Commit message: pcb layout
Parts:
- C36, C37, C38, C39, C42, C43, R3, R32, R33, R34, R35, R36, R47, R48, R49, R5, R50, R6, R7, R8: moved to B.Cu
- moved C37 18.8 mm to (152.9, 109.7)
- moved U5 14.0 mm to (152.4, 92.8), turned to 180 degrees
- moved R34 12.5 mm to (138.9, 90.4), turned to 180 degrees
- moved R35 11.2 mm to (135.8, 96.5)
- moved C32 10.8 mm to (170.2, 88.8)
- moved C33 10.8 mm to (169.9, 85.1)
- moved U10 10.8 mm to (169.7, 87.0)
- moved U6 10.2 mm to (152.4, 105.5), turned to 180 degrees
- moved U4 9.27 mm to (139.0, 93.5)
- moved R36 9.27 mm to (143.1, 93.7)
- moved R32 9.17 mm to (147.0, 104.9)
- moved R33 9.17 mm to (147.0, 101.5)
- moved C42 8.92 mm to (142.7, 116.3)
- moved R48 8.19 mm to (158.2, 110.2), turned to 270 degrees
- moved R6 7.06 mm to (183.1, 66.8), turned to 180 degrees
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Routing:
- net GND: track 0.00 -> 153.6 mm, vias 0 -> 19
- net /3V3_3: track 0.00 -> 84.7 mm, vias 0 -> 20
- net /SCL1: track 0.00 -> 66.1 mm, vias 0 -> 5
- net /SDA1: track 0.00 -> 62.1 mm, vias 0 -> 5
- net /sensors/3V3_2: track 0.00 -> 42.4 mm
- net Net-(D5-Pad2): track 0.00 -> 35.8 mm, vias 0 -> 2
- net Net-(C26-Pad2): track 0.00 -> 31.7 mm, vias 0 -> 2
- net Net-(D1-Pad1): track 0.00 -> 29.0 mm
- net Net-(C27-Pad1): track 0.00 -> 28.9 mm, vias 0 -> 2
- net /sensors/3V3_3: track 0.00 -> 27.8 mm, vias 0 -> 2
- net Net-(C28-Pad1): track 0.00 -> 27.0 mm, vias 0 -> 2
- net Net-(D10-Pad1): track 0.00 -> 26.9 mm, vias 0 -> 2
- net Net-(C26-Pad1): track 0.00 -> 26.9 mm, vias 0 -> 2
- net Net-(C27-Pad2): track 0.00 -> 26.3 mm, vias 0 -> 2
- net Net-(C29-Pad1): track 0.00 -> 23.4 mm, vias 0 -> 2
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- added copper zone on F.Cu, net /3V3_3
- added copper zone on B.Cu, net GND
Other:
- rule trace_min: 0.2 -> 0.15

Commit message: layout
Parts:
- moved FL2 44.5 mm to (129.5, 65.8)
- moved FL1 42.8 mm to (130.0, 109.0)
- moved R88 5.43 mm to (138.1, 103.0)
- moved R84 5.43 mm to (135.6, 103.0)
- moved R86 5.43 mm to (136.8, 103.0)
- moved R90 5.43 mm to (139.4, 103.0)
- moved R92 5.43 mm to (140.6, 103.0)
- moved R94 5.43 mm to (141.9, 103.0)
- moved R74 3.70 mm to (136.9, 96.8)
- moved R80 3.70 mm to (140.7, 96.9)
- moved R72 3.70 mm to (135.6, 96.8)
- moved R76 3.70 mm to (138.2, 96.8)
- moved R78 3.70 mm to (139.4, 96.8)
- moved R82 3.70 mm to (141.9, 96.9)
- moved R87 2.05 mm to (138.1, 91.1)
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Routing:
- net /mcu/OSC_IN: track 0.00 -> 9.66 mm, vias 0 -> 1
- net /mcu/OSC_OUT: track 0.00 -> 8.34 mm
- net Net-(C7-Pad1): track 0.00 -> 7.81 mm, vias 0 -> 1
- net Net-(R68-Pad2): track 0.00 -> 7.57 mm
- net /3V3_3: track 84.7 -> 91.8 mm, vias 20 -> 22
- net /ACC1: track 0.00 -> 6.73 mm
- net Net-(C6-Pad1): track 0.00 -> 6.66 mm, vias 0 -> 1
- net /3V3_1: track 6.36 -> 12.7 mm
- net GND: track 153.6 -> 158.7 mm, vias 19 -> 20
- net Net-(R58-Pad2): track 0.00 -> 5.03 mm
- net /ACC2: track 0.00 -> 4.55 mm
- net Net-(R61-Pad2): track 0.00 -> 4.53 mm
- net /FAULT2: track 0.00 -> 3.61 mm
- net /sensors/ASCL: track 0.00 -> 3.50 mm
- net Net-(R60-Pad2): track 0.00 -> 3.27 mm
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
Commit message: relayout
Parts:
- C23, C41, R34: moved to F.Cu
- C30, C31, C32, C33, C6, C7, C9, R10, R11, R4, R53, R55, R9, U10, U9, Y1: moved to B.Cu
- moved R97 85.4 mm to (228.7, 106.7)
- moved R98 85.4 mm to (231.0, 106.7)
- moved C36 83.9 mm to (234.7, 115.8)
- moved C37 83.9 mm to (234.7, 128.3)
- moved R32 83.9 mm to (228.7, 123.4)
- moved R33 83.9 mm to (228.7, 120.0)
- moved U5 83.9 mm to (234.2, 111.4)
- moved U6 83.9 mm to (234.2, 124.0)
- moved R49 82.9 mm to (237.3, 143.4)
- moved R50 82.9 mm to (237.3, 140.5)
- moved R68 82.6 mm to (65.3, 100.6)
- moved R47 82.4 mm to (237.5, 131.1)
- moved R48 82.4 mm to (237.2, 133.6)
- moved C29 81.4 mm to (263.7, 146.7)
- moved R43 81.4 mm to (263.4, 133.3)
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Routing:
- net GND: track 158.7 -> 0.00 mm, vias 20 -> 0
- net /3V3_3: track 91.8 -> 0.00 mm, vias 22 -> 0
- net /SCL1: track 66.1 -> 0.00 mm, vias 5 -> 0
- net /SDA1: track 62.1 -> 0.00 mm, vias 5 -> 0
- net /sensors/3V3_2: track 42.4 -> 0.00 mm
- net Net-(D5-Pad2): track 35.8 -> 0.00 mm, vias 2 -> 0
- net Net-(C26-Pad2): track 31.7 -> 0.00 mm, vias 2 -> 0
- net Net-(D1-Pad1): track 29.0 -> 0.00 mm
- net Net-(C27-Pad1): track 28.9 -> 0.00 mm, vias 2 -> 0
- net /sensors/3V3_3: track 27.8 -> 0.00 mm, vias 2 -> 0
- net Net-(C28-Pad1): track 27.0 -> 0.00 mm, vias 2 -> 0
- net Net-(D10-Pad1): track 26.9 -> 0.00 mm, vias 2 -> 0
- net Net-(C26-Pad1): track 26.9 -> 0.00 mm, vias 2 -> 0
- net Net-(C27-Pad2): track 26.3 -> 0.00 mm, vias 2 -> 0
- net Net-(C29-Pad1): track 23.4 -> 0.00 mm, vias 2 -> 0
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Other:
- net class Default: clearance 0.2 -> 0.11; via_dia 0.8 -> 0.6; via_drill 0.4 -> 0.3
- rule trace_clearance: 0.2 -> 0.11
- rule trace_min: 0.15 -> 0.11

Commit message: change layiut
Parts:
- C30, C31, C32, C33, R53, R55, U10, U9: moved to F.Cu
- moved R3 101.4 mm to (154.2, 125.5), turned to 0 degrees
- moved R97 96.4 mm to (160.7, 38.4)
- moved R98 96.4 mm to (162.9, 38.4)
- moved R31 88.6 mm to (186.4, 70.6), turned to 90 degrees
- moved L4 87.6 mm to (189.2, 71.4), turned to 90 degrees
- moved D4 84.9 mm to (179.3, 63.9)
- moved R23 84.9 mm to (174.3, 60.2)
- moved R25 84.9 mm to (176.3, 60.2)
- moved U5 84.9 mm to (165.1, 62.1)
- moved C36 84.9 mm to (165.6, 66.5)
- moved D2 84.9 mm to (173.0, 65.2)
- moved D7 84.9 mm to (181.6, 60.4)
- moved D8 84.9 mm to (179.4, 66.3)
- moved R29 84.9 mm to (171.4, 61.5)
- moved R24 84.7 mm to (175.7, 76.1)
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
Commit message: layout
Parts:
- C41, R12, R13, R14, R15, R16, R17: moved to B.Cu
- moved C41 90.0 mm to (151.9, 62.0), turned to 270 degrees
- moved R68 89.6 mm to (150.4, 72.6), turned to 180 degrees
- moved R69 83.9 mm to (150.4, 75.2)
- moved R67 82.8 mm to (139.2, 72.6)
- moved R70 82.5 mm to (150.4, 77.7), turned to 180 degrees
- moved R66 82.3 mm to (139.2, 75.2)
- moved R64 82.1 mm to (139.2, 79.8)
- moved R65 82.1 mm to (139.2, 77.2)
- moved U12 82.1 mm to (143.9, 76.2)
- moved R35 71.9 mm to (165.4, 104.4), turned to 270 degrees
- moved R95 69.9 mm to (167.1, 102.1), turned to 270 degrees
- moved R96 65.5 mm to (165.6, 99.1), turned to 0 degrees
- moved R84 65.5 mm to (140.8, 68.4), turned to 180 degrees
- moved U4 64.8 mm to (161.5, 102.5), turned to 90 degrees
- moved R86 64.6 mm to (140.8, 66.6), turned to 180 degrees
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Connections:
- J14 pad 17: /TX1 -> /TX4
- J14 pad 18: /TX2 -> /TX1
- J14 pad 19: /RX1 -> /RX4
- J14 pad 20: /RX2 -> /RX1
- J15 pad 17: /TX3 -> /TX2
- J15 pad 18: /TX4 -> /TX3
- J15 pad 19: /RX3 -> /RX2
- J15 pad 20: /RX4 -> /RX3
- L4 pad 2: Net-(L4-Pad2) -> Net-(D7-Pad2)
- R31 pad 2: Net-(L4-Pad2) -> Net-(D7-Pad2)
Routing:
- net Net-(D2-Pad1): track 0.00 -> 25.0 mm
- net Net-(D1-Pad1): track 0.00 -> 24.9 mm
- net Net-(D7-Pad2): track 0.00 -> 18.2 mm
- net Net-(D5-Pad2): track 0.00 -> 17.8 mm
- net Net-(J12-Pad2): track 0.00 -> 13.1 mm
- net Net-(J13-Pad2): track 0.00 -> 13.1 mm
- net Net-(J13-Pad1): track 0.00 -> 12.8 mm
- net Net-(J12-Pad1): track 0.00 -> 12.8 mm
- net /sensors/3V3_1: track 0.00 -> 8.60 mm
- net /sensors/3V3_3: track 0.00 -> 8.60 mm
- net Net-(J10-Pad2): track 0.00 -> 5.74 mm
- net Net-(J10-Pad1): track 0.00 -> 5.50 mm
- net Net-(J11-Pad2): track 0.00 -> 5.50 mm
- net Net-(J11-Pad1): track 0.00 -> 5.18 mm
- net Net-(D11-Pad2): track 0.00 -> 4.55 mm
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