File: obc_board/cubesat_obc.sch (KiCad schematic (older format))
At the start: 9 parts, among them J5 Conn_01x05_Female, J6 Conn_01x04_Female, J7 Conn_01x04_Female

Commit message: layout
Changed lines of the file:
@@
 $Descr A4 11693 8268
 encoding utf-8
-Sheet 1 7
+Sheet 1 8
 Title ""
 Date ""
@@
 F6 "SCK" I L 1400 3100 50
 F7 "CSB" I L 1400 3200 50
-F8 "SCL" I R 2750 2500 50
-F9 "SDA" I R 2750 2600 50
+F8 "SCL1" I R 2750 2500 50
+F9 "SDA1" I R 2750 2600 50
 F10 "ACC1" I R 2750 2900 50
 F11 "FAULT1" I R 2750 3000 50
@@
 Text Label 1450 1750 2    50   ~ 0
 SCK_3
-Text Label 8300 2350 2    50   ~ 0
-TX1
-Text Label 8300 2450 2    50   ~ 0
-RX1
-Text Label 8300 2650 2    50   ~ 0
-TX2
-Text Label 8300 2750 2    50   ~ 0
-RX2
-Text Label 8300 2950 2    50   ~ 0
-TX3
-Text Label 8300 3050 2    50   ~ 0
-RX3
-Text Label 5600 1450 0    50   ~ 0
-TX4
-Text Label 5600 1550 0    50   ~ 0
-RX4
-Text Label 5600 1750 0    50   ~ 0
-TX1
-Text Label 5600 1850 0    50   ~ 0
-RX1
-Text Label 8300 2150 2    50   ~ 0
-RX4
-Text Label 8300 2050 2    50   ~ 0
-TX4
 Text Label 10000 1650 0    50   ~ 0
 MISO_2
@@
 $EndComp
 $Sheet
-S 2050 4700 1700 1900
+S 1350 3950 1700 1900
 U 5F45B718
 F0 "stacking_connector" 50
 F1 "stacking_connector.sch" 50
-F2 "MISO" I R 3750 4950 50
-F3 "MOSI" I R 3750 5050 50
-F4 "SCK" I R 3750 5150 50
-F5 "CS1" I R 3750 5350 50
-F6 "CS2" I R 3750 5450 50
-F7 "TX1" I R 3750 5650 50
-F8 "RX1" I R 3750 5750 50
-F9 "TX2" I R 3750 5950 50
-F10 "RX2" I R 3750 6050 50
-F11 "SCL1" I L 2050 5950 50
-F12 "SDA1" I L 2050 6050 50
-F13 "SCL2" I L 2050 6250 50
-F14 "SDA2" I L 2050 6350 50
-F15 "3V3_P" I L 2050 4950 50
-F16 "GND" I L 2050 5700 50
-F17 "VBAT" I L 2050 5600 50
-F18 "3V3_1" I L 2050 5050 50
-F19 "3V3_2" I L 2050 5150 50
-F20 "VCC" I L 2050 5350 50
-F21 "3V3_3" I L 2050 5250 50
+F2 "MISO" I R 3050 4200 50
+F3 "MOSI" I R 3050 4300 50
+F4 "SCK" I R 3050 4400 50
+F5 "CS1" I R 3050 4600 50
+F6 "CS2" I R 3050 4700 50
+F7 "TX1" I R 3050 4900 50
+F8 "RX1" I R 3050 5000 50
+F9 "TX2" I R 3050 5200 50
+F10 "RX2" I R 3050 5300 50
+F11 "SCL1" I L 1350 5200 50
+F12 "SDA1" I L 1350 5300 50
+F13 "SCL2" I L 1350 5500 50
+F14 "SDA2" I L 1350 5600 50
+F15 "3V3_P" I L 1350 4200 50
+F16 "GND" I L 1350 4950 50
+F17 "VBAT" I L 1350 4850 50
+F18 "3V3_1" I L 1350 4300 50
+F19 "3V3_2" I L 1350 4400 50
+F20 "VCC" I L 1350 4600 50
+F21 "3V3_3" I L 1350 4500 50
 $EndSheet
-Text Label 2050 4950 2    50   ~ 0
+Text Label 1350 4200 2    50   ~ 0
 3V3_P
-Text Label 2050 5600 2    50   ~ 0
+Text Label 1350 4850 2    50   ~ 0
 VBAT
-Text Label 3750 5450 0    50   ~ 0
+Text Label 3050 4700 0    50   ~ 0
 CS2
-Text Label 3750 5350 0    50   ~ 0
+Text Label 3050 4600 0    50   ~ 0
 CS1
-Text Label 3750 5150 0    50   ~ 0
+Text Label 3050 4400 0    50   ~ 0
 SCK_2
-Text Label 3750 5050 0    50   ~ 0
+Text Label 3050 4300 0    50   ~ 0
 MOSI_2
-Text Label 3750 4950 0    50   ~ 0
+Text Label 3050 4200 0    50   ~ 0
 MISO_2
-Text Label 3750 5650 0    50   ~ 0
+Text Label 3050 4900 0    50   ~ 0
 TX4
-Text Label 3750 5750 0    50   ~ 0
+Text Label 3050 5000 0    50   ~ 0
 RX4
-Text Label 3750 6050 0    50   ~ 0
+Text Label 3050 5300 0    50   ~ 0
 RX3
-Text Label 3750 5950 0    50   ~ 0
+Text Label 3050 5200 0    50   ~ 0
 TX3
 $Comp
 L power:GND #PWR03
 U 1 1 5F33D67B
-P 1450 5850
-F 0 "#PWR03" H 1450 5600 50  0001 C CNN
-F 1 "GND" H 1455 5677 50  0000 C CNN
-F 2 "" H 1450 5850 50  0001 C CNN
-F 3 "" H 1450 5850 50  0001 C CNN
-	1    1450 5850
-	1    0    0    -1
-$EndComp
-Text Label 2050 6250 2    50   ~ 0
+P 750 5100
+F 0 "#PWR03" H 750 4850 50  0001 C CNN
+F 1 "GND" H 755 4927 50  0000 C CNN
+F 2 "" H 750 5100 50  0001 C CNN
+F 3 "" H 750 5100 50  0001 C CNN
+	1    750  5100
+	1    0    0    -1
+$EndComp
+Text Label 1350 5500 2    50   ~ 0
 SDA2
-Text Label 2050 6350 2    50   ~ 0
+Text Label 1350 5600 2    50   ~ 0
 SCL2
-Text Label 2050 6050 2    50   ~ 0
+Text Label 1350 5300 2    50   ~ 0
 SCL3
-Text Label 2050 5950 2    50   ~ 0
+Text Label 1350 5200 2    50   ~ 0
 SDA3
 Wire Wire Line
-	2050 5700 1450 5700
-Wire Wire Line
-	1450 5700 1450 5850
-Text Label 2050 5050 2    50   ~ 0
+	1350 4950 750  4950
+Wire Wire Line
+	750  4950 750  5100
+Text Label 1350 4300 2    50   ~ 0
 3V3_1
-Text Label 2050 5150 2    50   ~ 0
+Text Label 1350 4400 2    50   ~ 0
 3V3_2
-Text Label 2050 5250 2    50   ~ 0
+Text Label 1350 4500 2    50   ~ 0
 3V3_3
-Text Label 2050 5350 2    50   ~ 0
+Text Label 1350 4600 2    50   ~ 0
 VCC
 $Comp
@@
 CS2
 $Sheet
-S 4850 4700 1600 1900
+S 4150 3950 1600 1050
 U 5F6EB2F1
 F0 "uart_expander" 50
 F1 "uart_expander.sch" 50
-F2 "MISO" I R 6450 4950 50
-F3 "MOSI" I R 6450 5050 50
-F4 "SCK" I R 6450 5150 50
-F5 "RST" I R 6450 5350 50
-F6 "IRQ" I R 6450 5450 50
-F7 "CS" I R 6450 5550 50
-F8 "GND" I L 4850 5050 50
-F9 "3V3" I L 4850 4950 50
-F10 "VCC" I L 4850 5250 50
+F2 "MISO" I R 5750 4200 50
+F3 "MOSI" I R 5750 4300 50
+F4 "SCK" I R 5750 4400 50
+F5 "RST" I R 5750 4600 50
+F6 "IRQ" I R 5750 4700 50
+F7 "CS" I R 5750 4800 50
+F8 "GND" I L 4150 4300 50
+F9 "3V3" I L 4150 4200 50
+F10 "VCC" I L 4150 4500 50
 $EndSheet
-Text Label 5600 2150 0    50   ~ 0
-RX2
-Text Label 5600 2050 0    50   ~ 0
-TX2
-Text Label 5600 2350 0    50   ~ 0
-TX3
-Text Label 5600 2450 0    50   ~ 0
-RX3
 Text Label 8300 3500 2    50   ~ 0
 CS3
@@
 Text Label 8300 3200 2    50   ~ 0
 EXP
-Text Label 4850 5250 2    50   ~ 0
+Text Label 4150 4500 2    50   ~ 0
 VCC
-Text Label 4850 4950 2    50   ~ 0
+Text Label 4150 4200 2    50   ~ 0
 3V3_3
 $Comp
 L power:GND #PWR0101
 U 1 1 5F3B3184
-P 4500 5100
-F 0 "#PWR0101" H 4500 4850 50  0001 C CNN
-F 1 "GND" H 4505 4927 50  0000 C CNN
-F 2 "" H 4500 5100 50  0001 C CNN
-F 3 "" H 4500 5100 50  0001 C CNN
-	1    4500 5100
-	1    0    0    -1
-$EndComp
-Wire Wire Line
-	4850 5050 4500 5050
-Wire Wire Line
-	4500 5050 4500 5100
-Text Label 6450 5150 0    50   ~ 0
+P 3800 4350
+F 0 "#PWR0101" H 3800 4100 50  0001 C CNN
+F 1 "GND" H 3805 4177 50  0000 C CNN
+F 2 "" H 3800 4350 50  0001 C CNN
+F 3 "" H 3800 4350 50  0001 C CNN
+	1    3800 4350
+	1    0    0    -1
+$EndComp
+Wire Wire Line
+	4150 4300 3800 4300
+Wire Wire Line
+	3800 4300 3800 4350
+Text Label 5750 4400 0    50   ~ 0
 SCK_2
-Text Label 6450 5050 0    50   ~ 0
+Text Label 5750 4300 0    50   ~ 0
 MOSI_2
-Text Label 6450 4950 0    50   ~ 0
+Text Label 5750 4200 0    50   ~ 0
 MISO_2
-Text Label 6450 5550 0    50   ~ 0
+Text Label 5750 4800 0    50   ~ 0
 EXP
 Text Label 10000 3650 0    50   ~ 0
@@
 Text Label 10000 3750 0    50   ~ 0
 RST
-Text Label 6450 5350 0    50   ~ 0
+Text Label 5750 4600 0    50   ~ 0
 RST
-Text Label 6450 5450 0    50   ~ 0
+Text Label 5750 4700 0    50   ~ 0
 INT
+$Sheet
+S 4150 5450 1600 1150
+U 5F3F9D17
+F0 "ftdi" 50
+F1 "ftdi.sch" 50
+F2 "GND" I L 4150 5800 50
+F3 "RX1" I R 5750 5950 50
+F4 "TX1" I R 5750 5850 50
+F5 "RX0" I R 5750 5700 50
+F6 "TX0" I R 5750 5600 50
+F7 "RX2" I R 5750 6200 50
+F8 "TX2" I R 5750 6100 50
+F9 "TX3" I R 5750 6350 50
+F10 "RX3" I R 5750 6450 50
+$EndSheet
+$Comp
+L power:GND #PWR0102
+U 1 1 5F42F428
+P 3800 5850
+F 0 "#PWR0102" H 3800 5600 50  0001 C CNN
+F 1 "GND" H 3805 5677 50  0000 C CNN
+F 2 "" H 3800 5850 50  0001 C CNN
+F 3 "" H 3800 5850 50  0001 C CNN
+	1    3800 5850
+	1    0    0    -1
+$EndComp
+Wire Wire Line
+	4150 5800 3800 5800
+Wire Wire Line
+	3800 5800 3800 5850
+Text Label 5750 5600 0    50   ~ 0
+TX0
+Text Label 5750 5700 0    50   ~ 0
+RX0
+Text Label 5750 5850 0    50   ~ 0
+TX1
+Text Label 5750 5950 0    50   ~ 0
+RX1
+Text Label 5750 6100 0    50   ~ 0
+TX2
+Text Label 5750 6200 0    50   ~ 0
+RX2
+Text Label 5750 6350 0    50   ~ 0
+TX3
+Text Label 5750 6450 0    50   ~ 0
+RX3
+Text Label 5600 1450 0    50   ~ 0
+TX0
+Text Label 5600 1550 0    50   ~ 0
+RX0
+Text Label 5600 2050 0    50   ~ 0
+TX1
+Text Label 5600 2150 0    50   ~ 0
+RX1
+Text Label 8300 2150 2    50   ~ 0
+TX2
+Text Label 8300 2050 2    50   ~ 0
+RX2
+Text Label 5600 1750 0    50   ~ 0
+TX3
+Text Label 5600 1850 0    50   ~ 0
+RX3
 $EndSCHEMATC

Commit message: layout done
Parts:
- renumbered J5 to J1, J6 to J2, J7 to J3
Changed lines of the file:
@@
 $EndDescr
 $Comp
-L power:GND #PWR012
+L power:GND #PWR010
 U 1 1 5F33CD00
 P 7700 1450
-F 0 "#PWR012" H 7700 1200 50  0001 C CNN
+F 0 "#PWR010" H 7700 1200 50  0001 C CNN
 F 1 "GND" H 7705 1277 50  0000 C CNN
 F 2 "" H 7700 1450 50  0001 C CNN
@@
 	3650 1750 3650 1800
 $Comp
-L power:GND #PWR01
+L power:GND #PWR02
 U 1 1 5F33EB7E
 P 900 2650
-F 0 "#PWR01" H 900 2400 50  0001 C CNN
+F 0 "#PWR02" H 900 2400 50  0001 C CNN
 F 1 "GND" H 905 2477 50  0000 C CNN
 F 2 "" H 900 2650 50  0001 C CNN
@@
 RST2
 $Comp
-L power:GND #PWR02
+L power:GND #PWR03
 U 1 1 5F5192B7
 P 950 1400
-F 0 "#PWR02" H 950 1150 50  0001 C CNN
+F 0 "#PWR03" H 950 1150 50  0001 C CNN
 F 1 "GND" H 955 1227 50  0000 C CNN
 F 2 "" H 950 1400 50  0001 C CNN
@@
 SCK_2
 $Comp
-L Connector:Conn_01x04_Female J6
+L Connector:Conn_01x04_Female J2
 U 1 1 5F6F0159
 P 8050 5500
-F 0 "J6" H 8078 5476 50  0000 L CNN
+F 0 "J2" H 8078 5476 50  0000 L CNN
 F 1 "Conn_01x04_Female" H 8078 5385 50  0000 L CNN
 F 2 "Connector_Molex:Molex_PicoBlade_53261-0471_1x04-1MP_P1.25mm_Horizontal" H 8050 5500 50  0001 C CNN
@@
 ADC3
 $Comp
-L power:GND #PWR011
+L power:GND #PWR09
 U 1 1 5F6F2A66
 P 7600 5850
-F 0 "#PWR011" H 7600 5600 50  0001 C CNN
+F 0 "#PWR09" H 7600 5600 50  0001 C CNN
 F 1 "GND" H 7605 5677 50  0000 C CNN
 F 2 "" H 7600 5850 50  0001 C CNN
@@
 	7600 5700 7850 5700
 $Comp
-L Connector:Conn_01x04_Female J7
+L Connector:Conn_01x04_Female J3
 U 1 1 5F6F5054
 P 9500 5500
-F 0 "J7" H 9528 5476 50  0000 L CNN
+F 0 "J3" H 9528 5476 50  0000 L CNN
 F 1 "Conn_01x04_Female" H 9528 5385 50  0000 L CNN
 F 2 "Connector_Molex:Molex_PicoBlade_53261-0471_1x04-1MP_P1.25mm_Horizontal" H 9500 5500 50  0001 C CNN
@@
 $EndComp
 $Comp
-L power:GND #PWR013
+L power:GND #PWR011
 U 1 1 5F6F505D
 P 9050 5850
-F 0 "#PWR013" H 9050 5600 50  0001 C CNN
+F 0 "#PWR011" H 9050 5600 50  0001 C CNN
 F 1 "GND" H 9055 5677 50  0000 C CNN
 F 2 "" H 9050 5850 50  0001 C CNN
@@
 	7350 4400 7350 4450
 $Comp
-L power:GND #PWR010
+L power:GND #PWR08
 U 1 1 5F6FA8AC
 P 7350 4950
-F 0 "#PWR010" H 7350 4700 50  0001 C CNN
+F 0 "#PWR08" H 7350 4700 50  0001 C CNN
 F 1 "GND" H 7355 4777 50  0000 C CNN
 F 2 "" H 7350 4950 50  0001 C CNN
@@
 F5 "CS1" I R 3050 4600 50
 F6 "CS2" I R 3050 4700 50
-F7 "TX1" I R 3050 4900 50
-F8 "RX1" I R 3050 5000 50
-F9 "TX2" I R 3050 5200 50
-F10 "RX2" I R 3050 5300 50
-F11 "SCL1" I L 1350 5200 50
-F12 "SDA1" I L 1350 5300 50
-F13 "SCL2" I L 1350 5500 50
-F14 "SDA2" I L 1350 5600 50
-F15 "3V3_P" I L 1350 4200 50
-F16 "GND" I L 1350 4950 50
-F17 "VBAT" I L 1350 4850 50
-F18 "3V3_1" I L 1350 4300 50
-F19 "3V3_2" I L 1350 4400 50
-F20 "VCC" I L 1350 4600 50
-F21 "3V3_3" I L 1350 4500 50
+F7 "SCL1" I L 1350 5200 50
+F8 "SDA1" I L 1350 5300 50
+F9 "SCL2" I L 1350 5500 50
+F10 "SDA2" I L 1350 5600 50
+F11 "3V3_P" I L 1350 4200 50
+F12 "GND" I L 1350 4950 50
+F13 "VBAT" I L 1350 4850 50
+F14 "3V3_1" I L 1350 4300 50
+F15 "3V3_2" I L 1350 4400 50
+F16 "VCC" I L 1350 4600 50
+F17 "3V3_3" I L 1350 4500 50
 $EndSheet
 Text Label 1350 4200 2    50   ~ 0
@@
 Text Label 3050 4200 0    50   ~ 0
 MISO_2
-Text Label 3050 4900 0    50   ~ 0
-TX4
-Text Label 3050 5000 0    50   ~ 0
-RX4
-Text Label 3050 5300 0    50   ~ 0
-RX3
-Text Label 3050 5200 0    50   ~ 0
-TX3
-$Comp
-L power:GND #PWR03
+$Comp
+L power:GND #PWR01
 U 1 1 5F33D67B
 P 750 5100
-F 0 "#PWR03" H 750 4850 50  0001 C CNN
+F 0 "#PWR01" H 750 4850 50  0001 C CNN
 F 1 "GND" H 755 4927 50  0000 C CNN
 F 2 "" H 750 5100 50  0001 C CNN
@@
 VCC
 $Comp
-L power:GND #PWR09
+L power:GND #PWR07
 U 1 1 5F5B182E
 P 6250 3600
-F 0 "#PWR09" H 6250 3350 50  0001 C CNN
+F 0 "#PWR07" H 6250 3350 50  0001 C CNN
 F 1 "GND" H 6255 3427 50  0000 C CNN
 F 2 "" H 6250 3600 50  0001 C CNN
@@
 3V3_P
 $Comp
-L Connector:Conn_01x05_Female J5
+L Connector:Conn_01x05_Female J1
 U 1 1 5F3493AD
 P 6700 3250
-F 0 "J5" H 6728 3276 50  0000 L CNN
+F 0 "J1" H 6728 3276 50  0000 L CNN
 F 1 "Conn_01x05_Female" H 6728 3185 50  0000 L CNN
 F 2 "Connector_Molex:Molex_PicoBlade_53261-0571_1x05-1MP_P1.25mm_Horizontal" H 6700 3250 50  0001 C CNN
@@
 3V3_3
 $Comp
-L power:GND #PWR0101
+L power:GND #PWR05
 U 1 1 5F3B3184
 P 3800 4350
-F 0 "#PWR0101" H 3800 4100 50  0001 C CNN
+F 0 "#PWR05" H 3800 4100 50  0001 C CNN
 F 1 "GND" H 3805 4177 50  0000 C CNN
 F 2 "" H 3800 4350 50  0001 C CNN
@@
 $EndSheet
 $Comp
-L power:GND #PWR0102
+L power:GND #PWR06
 U 1 1 5F42F428
 P 3800 5850
-F 0 "#PWR0102" H 3800 5600 50  0001 C CNN
+F 0 "#PWR06" H 3800 5600 50  0001 C CNN
 F 1 "GND" H 3805 5677 50  0000 C CNN
 F 2 "" H 3800 5850 50  0001 C CNN
@@
 Text Label 5600 1850 0    50   ~ 0
 RX3
+Text Label 8300 2350 2    50   ~ 0
+TX1_OBC
+Text Label 8300 2450 2    50   ~ 0
+RX1_OBC
+Text Label 5600 2350 0    50   ~ 0
+TX1_OBC
+Text Label 5600 2450 0    50   ~ 0
+RX1_OBC
 $EndSCHEMATC

Commit message: relayout
Parts:
- added J1: Conn_01x08_Female, Connector_Molex:Molex_PicoBlade_53261-0871_1x08-1MP_P1.25mm_Horizontal, symbol Connector:Conn_01x08_Female
- renumbered J1 to J2, J2 to J3, J3 to J4
Connections:
- net 3V3_3: now also J1.2 (Pin_2)
- net ADC1: now also J3.2 (Pin_2); no longer J3.1 (Pin_1)
- net ADC2: now also J3.3 (Pin_3); no longer J3.2 (Pin_2)
- net ADC3: now also J3.4 (Pin_4); no longer J3.3 (Pin_3)
- net ADC4: now also J4.2 (Pin_2); no longer J4.1 (Pin_1)
- net ADC5: now also J4.3 (Pin_3); no longer J4.2 (Pin_2)
- net ADC6: now also J4.4 (Pin_4); no longer J4.3 (Pin_3)
- net CS3: now also J2.5 (Pin_5); no longer J2.4 (Pin_4)
- net GND: now also J2.1 (Pin_1), J3.1 (Pin_1), J4.1 (Pin_1), J1.1 (Pin_1); no longer J2.5 (Pin_5), J3.4 (Pin_4), J4.4 (Pin_4)
- net MISO_2: now also J2.4 (Pin_4); no longer J2.3 (Pin_3)
- net MOSI_2: now also J2.3 (Pin_3); no longer J2.2 (Pin_2)
- net SCK_2: now also J2.2 (Pin_2); no longer J2.1 (Pin_1)
- new net RX1_FTDI: J1.4 (Pin_4)
- new net RX2_FTDI: J1.6 (Pin_6)
- new net RX3_FTDI: J1.8 (Pin_8)
- new net TX1_FTDI: J1.3 (Pin_3)
- new net TX2_FTDI: J1.5 (Pin_5)
- new net TX3_FTDI: J1.7 (Pin_7)
Other:
- moved on the sheet: H1, H2, H3, H4, J2, J3, J4, R1, R2
