File: obc_board/modules.sch (KiCad schematic (older format))
At the start: 25 parts, among them J10 FSI-110-03-X-D-AD-SD-K-TR, J11 FSI-110-03-X-D-AD-SD-K-TR, J9 SAMTEC-MMS-110-01-X-DV, U12 LTC4304CMSTRPBF, U13 LTC4304CMSTRPBF

Commit message: expose more ios
Parts:
- removed C34: 10u, Capacitor_THT:CP_Radial_D5.0mm_P2.00mm, symbol Device:C
- removed FL1: PLT5BPH1015R6SNL, cubesat_obc:FIL_PLT5BPH1015R6SNL, symbol cubesat_obc_lib:PLT5BPH1015R6SNL
- removed J9: SAMTEC-MMS-110-01-X-DV, cubesat_obc:SAMTEC-MMS-110-01-X-DV, symbol cubesat_obc_lib:SAMTEC-MMS-110-01-X-DV
- added H? (x8): MountingHole, symbol Mechanical:MountingHole
Changed lines of the file:
@@
 $Descr A4 11693 8268
 encoding utf-8
-Sheet 5 5
+Sheet 5 6
 Title ""
 Date ""
@@
 UART1_TX
 $Comp
-L cubesat_obc_lib:SAMTEC-MMS-110-01-X-DV J9
-U 1 1 5FAC7ADC
-P 4050 5850
-F 0 "J9" H 4450 6117 50  0000 C CNN
-F 1 "SAMTEC-MMS-110-01-X-DV" H 4450 6026 50  0000 C CNN
-F 2 "cubesat_obc:SAMTEC-MMS-110-01-X-DV" H 4050 5850 50  0001 L BNN
-F 3 "https://www.digikey.sg/product-detail/en/samtec-inc/MMS-110-01-F-DV/MMS-110-01-F-DV-ND/7937063" H 4050 5850 50  0001 C CNN
-F 4 "MMS-110-01-F-DV-ND" H 4050 5850 50  0001 C CNN "Digikey Part Number"
-	1    4050 5850
-	1    0    0    -1
-$EndComp
-Text HLabel 1800 5850 0    50   Input ~ 0
-GND
-Text HLabel 1800 6250 0    50   Input ~ 0
-3V3_GPS
-Wire Wire Line
-	1800 6250 1900 6250
-$Comp
-L Device:C C34
-U 1 1 5FACB71A
-P 1900 6500
-F 0 "C34" H 2015 6546 50  0000 L CNN
-F 1 "10u" H 2015 6455 50  0000 L CNN
-F 2 "Capacitor_THT:CP_Radial_D5.0mm_P2.00mm" H 1938 6350 50  0001 C CNN
-F 3 "http://nichicon-us.com/english/products/pdfs/e-ukl.pdf~" H 1900 6500 50  0001 C CNN
-F 4 "493-13398-ND" H 1900 6500 50  0001 C CNN "Digikey Part Number"
-	1    1900 6500
-	1    0    0    -1
-$EndComp
-Wire Wire Line
-	1900 6250 1900 6350
-$Comp
-L cubesat_obc_lib:PLT5BPH1015R6SNL FL1
-U 1 1 5FACB726
-P 2350 6050
-F 0 "FL1" H 2350 6467 50  0000 C CNN
-F 1 "PLT5BPH1015R6SNL" H 2350 6376 50  0000 C CNN
-F 2 "cubesat_obc:FIL_PLT5BPH1015R6SNL" H 2350 6050 50  0001 L BNN
-F 3 "https://www.murata.com/en-us/products/productdata/8796762341406/QFLB9102.pdf" H 2350 6050 50  0001 L BNN
-F 4 "" H 2350 6050 50  0001 L BNN "Field4"
-F 5 "" H 2350 6050 50  0001 L BNN "Field5"
-F 6 "" H 2350 6050 50  0001 L BNN "Field6"
-F 7 "" H 2350 6050 50  0001 L BNN "Field7"
-F 8 "" H 2350 6050 50  0001 L BNN "Field8"
-F 9 "490-10976-1-ND" H 2350 6050 50  0001 C CNN "Digikey Part Number"
-	1    2350 6050
-	1    0    0    -1
-$EndComp
-Wire Wire Line
-	1800 5850 1950 5850
-Wire Wire Line
-	1900 6250 1950 6250
-Connection ~ 1900 6250
-Text HLabel 1900 6650 3    50   Input ~ 0
-GND
-Wire Wire Line
-	2750 5850 3000 5850
-Wire Wire Line
-	3000 5850 3000 6450
-Wire Wire Line
-	3000 6450 3850 6450
-Wire Wire Line
-	5050 6250 5700 6250
-Wire Wire Line
-	5700 6250 5700 6550
-Wire Wire Line
-	5700 7150 3000 7150
-Wire Wire Line
-	3000 7150 3000 6450
-Connection ~ 3000 6450
-Wire Wire Line
-	5050 6650 5700 6650
-Connection ~ 5700 6650
-Wire Wire Line
-	5700 6650 5700 7150
-Wire Wire Line
-	5100 6550 5700 6550
-Connection ~ 5700 6550
-Wire Wire Line
-	5700 6550 5700 6650
-Wire Wire Line
-	2750 6250 3100 6250
-Wire Wire Line
-	3100 6250 3100 5850
-Wire Wire Line
-	3100 5850 3850 5850
-Wire Wire Line
-	3100 6250 3100 7050
-Wire Wire Line
-	3100 7050 5600 7050
-Wire Wire Line
-	5600 7050 5600 5850
-Wire Wire Line
-	5600 5850 5050 5850
-Connection ~ 3100 6250
-Text HLabel 3850 6350 0    50   Input ~ 0
-GPS_TX
-Text HLabel 3850 6250 0    50   Input ~ 0
-GPS_TX3
-Text HLabel 3850 6550 0    50   Input ~ 0
-GPS_RX2
-Text HLabel 5050 6450 2    50   Input ~ 0
-GPS_TX2
-Text HLabel 5050 6350 2    50   Input ~ 0
-GPS_RX
-Text HLabel 5050 5950 2    50   Input ~ 0
-GPS_RX3
-Text HLabel 3850 6750 0    50   Input ~ 0
-PPS
-Text HLabel 5050 6050 2    50   Input ~ 0
-VARF
+L Mechanical:MountingHole H?
+U 1 1 5F3B0DB2
+P 6800 5800
+AR Path="/5F3B0DB2" Ref="H?"  Part="1"
+AR Path="/5FA4220C/5F3B0DB2" Ref="H?"  Part="1"
+F 0 "H?" H 6900 5846 50  0000 L CNN
+F 1 "MountingHole" H 6900 5755 50  0000 L CNN
+F 2 "" H 6800 5800 50  0001 C CNN
+F 3 "~" H 6800 5800 50  0001 C CNN
+	1    6800 5800
+	1    0    0    -1
+$EndComp
+$Comp
+L Mechanical:MountingHole H?
+U 1 1 5F3B0DB8
+P 6800 6000
+AR Path="/5F3B0DB8" Ref="H?"  Part="1"
+AR Path="/5FA4220C/5F3B0DB8" Ref="H?"  Part="1"
+F 0 "H?" H 6900 6046 50  0000 L CNN
+F 1 "MountingHole" H 6900 5955 50  0000 L CNN
+F 2 "" H 6800 6000 50  0001 C CNN
+F 3 "~" H 6800 6000 50  0001 C CNN
+	1    6800 6000
+	1    0    0    -1
+$EndComp
+$Comp
+L Mechanical:MountingHole H?
+U 1 1 5F3B0DBE
+P 6800 5600
+AR Path="/5F3B0DBE" Ref="H?"  Part="1"
+AR Path="/5FA4220C/5F3B0DBE" Ref="H?"  Part="1"
+F 0 "H?" H 6900 5646 50  0000 L CNN
+F 1 "MountingHole" H 6900 5555 50  0000 L CNN
+F 2 "" H 6800 5600 50  0001 C CNN
+F 3 "~" H 6800 5600 50  0001 C CNN
+	1    6800 5600
+	1    0    0    -1
+$EndComp
+$Comp
+L Mechanical:MountingHole H?
+U 1 1 5F3B0DC4
+P 6800 5400
+AR Path="/5F3B0DC4" Ref="H?"  Part="1"
+AR Path="/5FA4220C/5F3B0DC4" Ref="H?"  Part="1"
+F 0 "H?" H 6900 5446 50  0000 L CNN
+F 1 "MountingHole" H 6900 5355 50  0000 L CNN
+F 2 "" H 6800 5400 50  0001 C CNN
+F 3 "~" H 6800 5400 50  0001 C CNN
+	1    6800 5400
+	1    0    0    -1
+$EndComp
+$Comp
+L Mechanical:MountingHole H?
+U 1 1 5F3B5CFB
+P 7600 5800
+AR Path="/5F3B5CFB" Ref="H?"  Part="1"
+AR Path="/5FA4220C/5F3B5CFB" Ref="H?"  Part="1"
+F 0 "H?" H 7700 5846 50  0000 L CNN
+F 1 "MountingHole" H 7700 5755 50  0000 L CNN
+F 2 "" H 7600 5800 50  0001 C CNN
+F 3 "~" H 7600 5800 50  0001 C CNN
+	1    7600 5800
+	1    0    0    -1
+$EndComp
+$Comp
+L Mechanical:MountingHole H?
+U 1 1 5F3B5D01
+P 7600 6000
+AR Path="/5F3B5D01" Ref="H?"  Part="1"
+AR Path="/5FA4220C/5F3B5D01" Ref="H?"  Part="1"
+F 0 "H?" H 7700 6046 50  0000 L CNN
+F 1 "MountingHole" H 7700 5955 50  0000 L CNN
+F 2 "" H 7600 6000 50  0001 C CNN
+F 3 "~" H 7600 6000 50  0001 C CNN
+	1    7600 6000
+	1    0    0    -1
+$EndComp
+$Comp
+L Mechanical:MountingHole H?
+U 1 1 5F3B5D07
+P 7600 5600
+AR Path="/5F3B5D07" Ref="H?"  Part="1"
+AR Path="/5FA4220C/5F3B5D07" Ref="H?"  Part="1"
+F 0 "H?" H 7700 5646 50  0000 L CNN
+F 1 "MountingHole" H 7700 5555 50  0000 L CNN
+F 2 "" H 7600 5600 50  0001 C CNN
+F 3 "~" H 7600 5600 50  0001 C CNN
+	1    7600 5600
+	1    0    0    -1
+$EndComp
+$Comp
+L Mechanical:MountingHole H?
+U 1 1 5F3B5D0D
+P 7600 5400
+AR Path="/5F3B5D0D" Ref="H?"  Part="1"
+AR Path="/5FA4220C/5F3B5D0D" Ref="H?"  Part="1"
+F 0 "H?" H 7700 5446 50  0000 L CNN
+F 1 "MountingHole" H 7700 5355 50  0000 L CNN
+F 2 "" H 7600 5400 50  0001 C CNN
+F 3 "~" H 7600 5400 50  0001 C CNN
+	1    7600 5400
+	1    0    0    -1
+$EndComp
 $EndSCHEMATC

Commit message: pcb layout
Parts:
- C34: renamed from C35; footprint Capacitor_THT:CP_Radial_D5.0mm_P2.00mm -> Capacitor_SMD:CP_Elec_4x5.3; Digikey Part Number 493-13398-ND -> 565-2442-1-ND
- C35: renamed from C36; footprint Capacitor_THT:CP_Radial_D5.0mm_P2.00mm -> Capacitor_SMD:CP_Elec_4x5.3; Digikey Part Number 493-13398-ND -> 565-2442-1-ND
- H10, H11, H12, H5, H6, H7, H8, H9: renamed from H?; footprint (none) -> Mounting_Wuerth:Mounting_Wuerth_WA-SMSI-M3_H3mm_9774030360; Digikey Part Number (none) -> 732-5270-1-ND; Field4 (none) -> 732-5270-1-ND
- renumbered FL2 to FL1, FL3 to FL2, J10 to J14, J11 to J15, R56 to R57, R57 to R58, R58 to R59, R59 to R60, R60 to R61, R61 to R62, R62 to R63, R63 to R64, R64 to R65, R65 to R66, R66 to R67, R67 to R68, R68 to R69, R69 to R70, U12 to U11, U13 to U12

Commit message: layout
Connections:
- net UART0_RX: no longer J15.17
- net UART0_TX: no longer J15.19
- net UART1_RX: no longer J15.18
- net UART1_TX: no longer J15.20
- new net UART2_RX: J15.17
- new net UART2_TX: J15.19
- new net UART3_RX: J15.18
- new net UART3_TX: J15.20
Changed lines of the file:
@@
 	9450 2700 9350 2700
 Text HLabel 8350 3300 0    50   Input ~ 0
-UART0_RX
+UART2_RX
 Wire Wire Line
 	6850 2900 8350 2900
@@
 	7600 1900 9750 1900
 Text HLabel 8350 3400 0    50   Input ~ 0
-UART0_TX
+UART2_TX
 Text HLabel 9350 3300 2    50   Input ~ 0
-UART1_RX
+UART3_RX
 Text HLabel 9350 3400 2    50   Input ~ 0
-UART1_TX
+UART3_TX
 $Comp
 L Mechanical:MountingHole H?

Commit message: layout done
Parts:
- renumbered C34 to C38, C35 to C39, J14 to J10, J15 to J11, R57 to R55, R58 to R56, R59 to R57, R60 to R58, R61 to R59, R62 to R60, R63 to R61, R64 to R62, R65 to R63, R66 to R64, R67 to R65, R68 to R66, R69 to R67, R70 to R68
Changed lines of the file:
@@
 $EndDescr
 $Comp
-L cubesat_obc_lib:FSI-110-03-X-D-AD-SD-K-TR J14
+L cubesat_obc_lib:FSI-110-03-X-D-AD-SD-K-TR J10
 U 1 1 5FA42BE1
 P 4550 3000
-F 0 "J14" H 4550 3767 50  0000 C CNN
+F 0 "J10" H 4550 3767 50  0000 C CNN
 F 1 "FSI-110-03-X-D-AD-SD-K-TR" H 4550 3676 50  0000 C CNN
 F 2 "cubesat_obc:SAMTEC_FSI-110-10-X-D-AD-TR" H 4550 3000 50  0001 L BNN
@@
 	2150 2700 2250 2700
 $Comp
-L Device:C C34
+L Device:C C38
 U 1 1 5FA44CB1
 P 2250 2950
-F 0 "C34" H 2365 2996 50  0000 L CNN
+F 0 "C38" H 2365 2996 50  0000 L CNN
 F 1 "10u" H 2365 2905 50  0000 L CNN
 F 2 "Capacitor_SMD:CP_Elec_4x5.3" H 2288 2800 50  0001 C CNN
@@
 P 3000 3950
 AR Path="/5F315FB6/5FA51731" Ref="R?"  Part="1"
-AR Path="/5FA4220C/5FA51731" Ref="R60"  Part="1"
-F 0 "R60" H 3070 3996 50  0000 L CNN
+AR Path="/5FA4220C/5FA51731" Ref="R58"  Part="1"
+F 0 "R58" H 3070 3996 50  0000 L CNN
 F 1 "10k" H 3070 3905 50  0000 L CNN
 F 2 "Resistor_SMD:R_0402_1005Metric" V 2930 3950 50  0001 C CNN
@@
 P 2250 4100
 AR Path="/5F315FB6/5FA5173F" Ref="R?"  Part="1"
-AR Path="/5FA4220C/5FA5173F" Ref="R57"  Part="1"
-F 0 "R57" H 2320 4146 50  0000 L CNN
+AR Path="/5FA4220C/5FA5173F" Ref="R55"  Part="1"
+F 0 "R55" H 2320 4146 50  0000 L CNN
 F 1 "10k" H 2320 4055 50  0000 L CNN
 F 2 "Resistor_SMD:R_0402_1005Metric" V 2180 4100 50  0001 C CNN
@@
 P 4750 4100
 AR Path="/5F315FB6/5FA5174A" Ref="R?"  Part="1"
-AR Path="/5FA4220C/5FA5174A" Ref="R63"  Part="1"
-F 0 "R63" H 4820 4146 50  0000 L CNN
+AR Path="/5FA4220C/5FA5174A" Ref="R61"  Part="1"
+F 0 "R61" H 4820 4146 50  0000 L CNN
 F 1 "10k" H 4820 4055 50  0000 L CNN
 F 2 "Resistor_SMD:R_0402_1005Metric" V 4680 4100 50  0001 C CNN
@@
 P 3450 3650
 AR Path="/5F315FB6/5FA5ADB3" Ref="R?"  Part="1"
-AR Path="/5FA4220C/5FA5ADB3" Ref="R62"  Part="1"
-F 0 "R62" H 3520 3696 50  0000 L CNN
+AR Path="/5FA4220C/5FA5ADB3" Ref="R60"  Part="1"
+F 0 "R60" H 3520 3696 50  0000 L CNN
 F 1 "10k" H 3520 3605 50  0000 L CNN
 F 2 "Resistor_SMD:R_0402_1005Metric" V 3380 3650 50  0001 C CNN
@@
 P 2700 3950
 AR Path="/5F315FB6/5FA5BDA5" Ref="R?"  Part="1"
-AR Path="/5FA4220C/5FA5BDA5" Ref="R59"  Part="1"
-F 0 "R59" H 2770 3996 50  0000 L CNN
+AR Path="/5FA4220C/5FA5BDA5" Ref="R57"  Part="1"
+F 0 "R57" H 2770 3996 50  0000 L CNN
 F 1 "10k" H 2770 3905 50  0000 L CNN
 F 2 "Resistor_SMD:R_0402_1005Metric" V 2630 3950 50  0001 C CNN
@@
 P 2550 3300
 AR Path="/5F315FB6/5FA7F305" Ref="R?"  Part="1"
-AR Path="/5FA4220C/5FA7F305" Ref="R58"  Part="1"
-F 0 "R58" H 2620 3346 50  0000 L CNN
+AR Path="/5FA4220C/5FA7F305" Ref="R56"  Part="1"
+F 0 "R56" H 2620 3346 50  0000 L CNN
 F 1 "1k" H 2620 3255 50  0000 L CNN
 F 2 "Resistor_SMD:R_0402_1005Metric" V 2480 3300 50  0001 C CNN
@@
 P 3150 3300
 AR Path="/5F315FB6/5FA89462" Ref="R?"  Part="1"
-AR Path="/5FA4220C/5FA89462" Ref="R61"  Part="1"
-F 0 "R61" H 3220 3346 50  0000 L CNN
+AR Path="/5FA4220C/5FA89462" Ref="R59"  Part="1"
+F 0 "R59" H 3220 3346 50  0000 L CNN
 F 1 "1k" H 3220 3255 50  0000 L CNN
 F 2 "Resistor_SMD:R_0402_1005Metric" V 3080 3300 50  0001 C CNN
@@
 UART1_TX
 $Comp
-L cubesat_obc_lib:FSI-110-03-X-D-AD-SD-K-TR J15
+L cubesat_obc_lib:FSI-110-03-X-D-AD-SD-K-TR J11
 U 1 1 5FAAED71
 P 8850 3000
-F 0 "J15" H 8850 3767 50  0000 C CNN
+F 0 "J11" H 8850 3767 50  0000 C CNN
 F 1 "FSI-110-03-X-D-AD-SD-K-TR" H 8850 3676 50  0000 C CNN
 F 2 "cubesat_obc:SAMTEC_FSI-110-10-X-D-AD-TR" H 8850 3000 50  0001 L BNN
@@
 	6450 2700 6550 2700
 $Comp
-L Device:C C35
+L Device:C C39
 U 1 1 5FAAED7A
 P 6550 2950
-F 0 "C35" H 6665 2996 50  0000 L CNN
+F 0 "C39" H 6665 2996 50  0000 L CNN
 F 1 "10u" H 6665 2905 50  0000 L CNN
 F 2 "Capacitor_SMD:CP_Elec_4x5.3" H 6588 2800 50  0001 C CNN
@@
 P 7300 3950
 AR Path="/5F315FB6/5FAAED9A" Ref="R?"  Part="1"
-AR Path="/5FA4220C/5FAAED9A" Ref="R67"  Part="1"
-F 0 "R67" H 7370 3996 50  0000 L CNN
+AR Path="/5FA4220C/5FAAED9A" Ref="R65"  Part="1"
+F 0 "R65" H 7370 3996 50  0000 L CNN
 F 1 "10k" H 7370 3905 50  0000 L CNN
 F 2 "Resistor_SMD:R_0402_1005Metric" V 7230 3950 50  0001 C CNN
@@
 P 6550 4100
 AR Path="/5F315FB6/5FAAEDA8" Ref="R?"  Part="1"
-AR Path="/5FA4220C/5FAAEDA8" Ref="R64"  Part="1"
-F 0 "R64" H 6620 4146 50  0000 L CNN
+AR Path="/5FA4220C/5FAAEDA8" Ref="R62"  Part="1"
+F 0 "R62" H 6620 4146 50  0000 L CNN
 F 1 "10k" H 6620 4055 50  0000 L CNN
 F 2 "Resistor_SMD:R_0402_1005Metric" V 6480 4100 50  0001 C CNN
@@
 P 9050 4100
 AR Path="/5F315FB6/5FAAEDB2" Ref="R?"  Part="1"
-AR Path="/5FA4220C/5FAAEDB2" Ref="R70"  Part="1"
-F 0 "R70" H 9120 4146 50  0000 L CNN
+AR Path="/5FA4220C/5FAAEDB2" Ref="R68"  Part="1"
+F 0 "R68" H 9120 4146 50  0000 L CNN
 F 1 "10k" H 9120 4055 50  0000 L CNN
 F 2 "Resistor_SMD:R_0402_1005Metric" V 8980 4100 50  0001 C CNN
@@
 P 7750 3650
 AR Path="/5F315FB6/5FAAEDC2" Ref="R?"  Part="1"
-AR Path="/5FA4220C/5FAAEDC2" Ref="R69"  Part="1"
-F 0 "R69" H 7820 3696 50  0000 L CNN
+AR Path="/5FA4220C/5FAAEDC2" Ref="R67"  Part="1"
+F 0 "R67" H 7820 3696 50  0000 L CNN
 F 1 "10k" H 7820 3605 50  0000 L CNN
 F 2 "Resistor_SMD:R_0402_1005Metric" V 7680 3650 50  0001 C CNN
@@
 P 7000 3950
 AR Path="/5F315FB6/5FAAEDCA" Ref="R?"  Part="1"
-AR Path="/5FA4220C/5FAAEDCA" Ref="R66"  Part="1"
-F 0 "R66" H 7070 3996 50  0000 L CNN
+AR Path="/5FA4220C/5FAAEDCA" Ref="R64"  Part="1"
+F 0 "R64" H 7070 3996 50  0000 L CNN
 F 1 "10k" H 7070 3905 50  0000 L CNN
 F 2 "Resistor_SMD:R_0402_1005Metric" V 6930 3950 50  0001 C CNN
@@
 P 6850 3300
 AR Path="/5F315FB6/5FAAEDD8" Ref="R?"  Part="1"
-AR Path="/5FA4220C/5FAAEDD8" Ref="R65"  Part="1"
-F 0 "R65" H 6920 3346 50  0000 L CNN
+AR Path="/5FA4220C/5FAAEDD8" Ref="R63"  Part="1"
+F 0 "R63" H 6920 3346 50  0000 L CNN
 F 1 "1k" H 6920 3255 50  0000 L CNN
 F 2 "Resistor_SMD:R_0402_1005Metric" V 6780 3300 50  0001 C CNN
@@
 P 7450 3300
 AR Path="/5F315FB6/5FAAEDE1" Ref="R?"  Part="1"
-AR Path="/5FA4220C/5FAAEDE1" Ref="R68"  Part="1"
-F 0 "R68" H 7520 3346 50  0000 L CNN
+AR Path="/5FA4220C/5FAAEDE1" Ref="R66"  Part="1"
+F 0 "R66" H 7520 3346 50  0000 L CNN
 F 1 "1k" H 7520 3255 50  0000 L CNN
 F 2 "Resistor_SMD:R_0402_1005Metric" V 7380 3300 50  0001 C CNN
