File: obc_board/modules.sch (KiCad schematic (older format))
At the start: 30 parts, among them J10 FSI-110-03-X-D-AD-SD-K-TR, J11 FSI-110-03-X-D-AD-SD-K-TR, U11 LTC4304CMSTRPBF, U12 LTC4304CMSTRPBF

Commit message: relayout
Parts:
- C33: renamed from C38; footprint Capacitor_SMD:CP_Elec_4x5.3 -> Capacitor_SMD:C_1206_3216Metric; Digikey Part Number 565-2442-1-ND -> 311-1952-1-ND
- C34: renamed from C39; footprint Capacitor_SMD:CP_Elec_4x5.3 -> Capacitor_SMD:C_1206_3216Metric; Digikey Part Number 565-2442-1-ND -> 311-1952-1-ND
- renumbered J11 to J10, J10 to J9, R55 to R48, R56 to R49, R57 to R50, R58 to R51, R59 to R52, R60 to R53, R61 to R54, R62 to R55, R63 to R56, R64 to R57, R65 to R58, R66 to R59, R67 to R60, R68 to R61
Changed lines of the file:
@@
 $Descr A4 11693 8268
 encoding utf-8
-Sheet 5 8
+Sheet 4 8
 Title ""
 Date ""
@@
 $EndDescr
 $Comp
-L cubesat_obc_lib:FSI-110-03-X-D-AD-SD-K-TR J10
+L cubesat_obc_lib:FSI-110-03-X-D-AD-SD-K-TR J9
 U 1 1 5FA42BE1
 P 4550 3000
-F 0 "J10" H 4550 3767 50  0000 C CNN
+F 0 "J9" H 4550 3767 50  0000 C CNN
 F 1 "FSI-110-03-X-D-AD-SD-K-TR" H 4550 3676 50  0000 C CNN
 F 2 "cubesat_obc:SAMTEC_FSI-110-10-X-D-AD-TR" H 4550 3000 50  0001 L BNN
@@
 	2150 2700 2250 2700
 $Comp
-L Device:C C38
+L Device:C C33
 U 1 1 5FA44CB1
 P 2250 2950
-F 0 "C38" H 2365 2996 50  0000 L CNN
+F 0 "C33" H 2365 2996 50  0000 L CNN
 F 1 "10u" H 2365 2905 50  0000 L CNN
-F 2 "Capacitor_SMD:CP_Elec_4x5.3" H 2288 2800 50  0001 C CNN
-F 3 "http://www.chemi-con.co.jp/cgi-bin/CAT_DB/SEARCH/cat_db_al.cgi?e=e&j=p&pdfname=mvy" H 2250 2950 50  0001 C CNN
-F 4 "565-2442-1-ND" H 2250 2950 50  0001 C CNN "Digikey Part Number"
+F 2 "Capacitor_SMD:C_1206_3216Metric" H 2288 2800 50  0001 C CNN
+F 3 "https://www.yageo.com/upload/media/product/productsearch/datasheet/mlcc/UPY-GPHC_X7R_6.3V-to-50V_18.pdf" H 2250 2950 50  0001 C CNN
+F 4 "311-1952-1-ND" H 2250 2950 50  0001 C CNN "Digikey Part Number"
 	1    2250 2950
 	1    0    0    -1
@@
 P 3000 3950
 AR Path="/5F315FB6/5FA51731" Ref="R?"  Part="1"
-AR Path="/5FA4220C/5FA51731" Ref="R58"  Part="1"
-F 0 "R58" H 3070 3996 50  0000 L CNN
+AR Path="/5FA4220C/5FA51731" Ref="R51"  Part="1"
+F 0 "R51" H 3070 3996 50  0000 L CNN
 F 1 "10k" H 3070 3905 50  0000 L CNN
 F 2 "Resistor_SMD:R_0402_1005Metric" V 2930 3950 50  0001 C CNN
@@
 P 2250 4100
 AR Path="/5F315FB6/5FA5173F" Ref="R?"  Part="1"
-AR Path="/5FA4220C/5FA5173F" Ref="R55"  Part="1"
-F 0 "R55" H 2320 4146 50  0000 L CNN
+AR Path="/5FA4220C/5FA5173F" Ref="R48"  Part="1"
+F 0 "R48" H 2320 4146 50  0000 L CNN
 F 1 "10k" H 2320 4055 50  0000 L CNN
 F 2 "Resistor_SMD:R_0402_1005Metric" V 2180 4100 50  0001 C CNN
@@
 P 4750 4100
 AR Path="/5F315FB6/5FA5174A" Ref="R?"  Part="1"
-AR Path="/5FA4220C/5FA5174A" Ref="R61"  Part="1"
-F 0 "R61" H 4820 4146 50  0000 L CNN
+AR Path="/5FA4220C/5FA5174A" Ref="R54"  Part="1"
+F 0 "R54" H 4820 4146 50  0000 L CNN
 F 1 "10k" H 4820 4055 50  0000 L CNN
 F 2 "Resistor_SMD:R_0402_1005Metric" V 4680 4100 50  0001 C CNN
@@
 P 3450 3650
 AR Path="/5F315FB6/5FA5ADB3" Ref="R?"  Part="1"
-AR Path="/5FA4220C/5FA5ADB3" Ref="R60"  Part="1"
-F 0 "R60" H 3520 3696 50  0000 L CNN
+AR Path="/5FA4220C/5FA5ADB3" Ref="R53"  Part="1"
+F 0 "R53" H 3520 3696 50  0000 L CNN
 F 1 "10k" H 3520 3605 50  0000 L CNN
 F 2 "Resistor_SMD:R_0402_1005Metric" V 3380 3650 50  0001 C CNN
@@
 P 2700 3950
 AR Path="/5F315FB6/5FA5BDA5" Ref="R?"  Part="1"
-AR Path="/5FA4220C/5FA5BDA5" Ref="R57"  Part="1"
-F 0 "R57" H 2770 3996 50  0000 L CNN
+AR Path="/5FA4220C/5FA5BDA5" Ref="R50"  Part="1"
+F 0 "R50" H 2770 3996 50  0000 L CNN
 F 1 "10k" H 2770 3905 50  0000 L CNN
 F 2 "Resistor_SMD:R_0402_1005Metric" V 2630 3950 50  0001 C CNN
@@
 P 2550 3300
 AR Path="/5F315FB6/5FA7F305" Ref="R?"  Part="1"
-AR Path="/5FA4220C/5FA7F305" Ref="R56"  Part="1"
-F 0 "R56" H 2620 3346 50  0000 L CNN
+AR Path="/5FA4220C/5FA7F305" Ref="R49"  Part="1"
+F 0 "R49" H 2620 3346 50  0000 L CNN
 F 1 "1k" H 2620 3255 50  0000 L CNN
 F 2 "Resistor_SMD:R_0402_1005Metric" V 2480 3300 50  0001 C CNN
@@
 P 3150 3300
 AR Path="/5F315FB6/5FA89462" Ref="R?"  Part="1"
-AR Path="/5FA4220C/5FA89462" Ref="R59"  Part="1"
-F 0 "R59" H 3220 3346 50  0000 L CNN
+AR Path="/5FA4220C/5FA89462" Ref="R52"  Part="1"
+F 0 "R52" H 3220 3346 50  0000 L CNN
 F 1 "1k" H 3220 3255 50  0000 L CNN
 F 2 "Resistor_SMD:R_0402_1005Metric" V 3080 3300 50  0001 C CNN
@@
 UART1_TX
 $Comp
-L cubesat_obc_lib:FSI-110-03-X-D-AD-SD-K-TR J11
+L cubesat_obc_lib:FSI-110-03-X-D-AD-SD-K-TR J10
 U 1 1 5FAAED71
 P 8850 3000
-F 0 "J11" H 8850 3767 50  0000 C CNN
+F 0 "J10" H 8850 3767 50  0000 C CNN
 F 1 "FSI-110-03-X-D-AD-SD-K-TR" H 8850 3676 50  0000 C CNN
 F 2 "cubesat_obc:SAMTEC_FSI-110-10-X-D-AD-TR" H 8850 3000 50  0001 L BNN
@@
 	6450 2700 6550 2700
 $Comp
-L Device:C C39
+L Device:C C34
 U 1 1 5FAAED7A
 P 6550 2950
-F 0 "C39" H 6665 2996 50  0000 L CNN
+F 0 "C34" H 6665 2996 50  0000 L CNN
 F 1 "10u" H 6665 2905 50  0000 L CNN
-F 2 "Capacitor_SMD:CP_Elec_4x5.3" H 6588 2800 50  0001 C CNN
-F 3 "http://www.chemi-con.co.jp/cgi-bin/CAT_DB/SEARCH/cat_db_al.cgi?e=e&j=p&pdfname=mvy" H 6550 2950 50  0001 C CNN
-F 4 "565-2442-1-ND" H 6550 2950 50  0001 C CNN "Digikey Part Number"
+F 2 "Capacitor_SMD:C_1206_3216Metric" H 6588 2800 50  0001 C CNN
+F 3 "https://www.yageo.com/upload/media/product/productsearch/datasheet/mlcc/UPY-GPHC_X7R_6.3V-to-50V_18.pdf" H 6550 2950 50  0001 C CNN
+F 4 "311-1952-1-ND" H 6550 2950 50  0001 C CNN "Digikey Part Number"
 	1    6550 2950
 	1    0    0    -1
@@
 P 7300 3950
 AR Path="/5F315FB6/5FAAED9A" Ref="R?"  Part="1"
-AR Path="/5FA4220C/5FAAED9A" Ref="R65"  Part="1"
-F 0 "R65" H 7370 3996 50  0000 L CNN
+AR Path="/5FA4220C/5FAAED9A" Ref="R58"  Part="1"
+F 0 "R58" H 7370 3996 50  0000 L CNN
 F 1 "10k" H 7370 3905 50  0000 L CNN
 F 2 "Resistor_SMD:R_0402_1005Metric" V 7230 3950 50  0001 C CNN
@@
 P 6550 4100
 AR Path="/5F315FB6/5FAAEDA8" Ref="R?"  Part="1"
-AR Path="/5FA4220C/5FAAEDA8" Ref="R62"  Part="1"
-F 0 "R62" H 6620 4146 50  0000 L CNN
+AR Path="/5FA4220C/5FAAEDA8" Ref="R55"  Part="1"
+F 0 "R55" H 6620 4146 50  0000 L CNN
 F 1 "10k" H 6620 4055 50  0000 L CNN
 F 2 "Resistor_SMD:R_0402_1005Metric" V 6480 4100 50  0001 C CNN
@@
 P 9050 4100
 AR Path="/5F315FB6/5FAAEDB2" Ref="R?"  Part="1"
-AR Path="/5FA4220C/5FAAEDB2" Ref="R68"  Part="1"
-F 0 "R68" H 9120 4146 50  0000 L CNN
+AR Path="/5FA4220C/5FAAEDB2" Ref="R61"  Part="1"
+F 0 "R61" H 9120 4146 50  0000 L CNN
 F 1 "10k" H 9120 4055 50  0000 L CNN
 F 2 "Resistor_SMD:R_0402_1005Metric" V 8980 4100 50  0001 C CNN
@@
 P 7750 3650
 AR Path="/5F315FB6/5FAAEDC2" Ref="R?"  Part="1"
-AR Path="/5FA4220C/5FAAEDC2" Ref="R67"  Part="1"
-F 0 "R67" H 7820 3696 50  0000 L CNN
+AR Path="/5FA4220C/5FAAEDC2" Ref="R60"  Part="1"
+F 0 "R60" H 7820 3696 50  0000 L CNN
 F 1 "10k" H 7820 3605 50  0000 L CNN
 F 2 "Resistor_SMD:R_0402_1005Metric" V 7680 3650 50  0001 C CNN
@@
 P 7000 3950
 AR Path="/5F315FB6/5FAAEDCA" Ref="R?"  Part="1"
-AR Path="/5FA4220C/5FAAEDCA" Ref="R64"  Part="1"
-F 0 "R64" H 7070 3996 50  0000 L CNN
+AR Path="/5FA4220C/5FAAEDCA" Ref="R57"  Part="1"
+F 0 "R57" H 7070 3996 50  0000 L CNN
 F 1 "10k" H 7070 3905 50  0000 L CNN
 F 2 "Resistor_SMD:R_0402_1005Metric" V 6930 3950 50  0001 C CNN
@@
 P 6850 3300
 AR Path="/5F315FB6/5FAAEDD8" Ref="R?"  Part="1"
-AR Path="/5FA4220C/5FAAEDD8" Ref="R63"  Part="1"
-F 0 "R63" H 6920 3346 50  0000 L CNN
+AR Path="/5FA4220C/5FAAEDD8" Ref="R56"  Part="1"
+F 0 "R56" H 6920 3346 50  0000 L CNN
 F 1 "1k" H 6920 3255 50  0000 L CNN
 F 2 "Resistor_SMD:R_0402_1005Metric" V 6780 3300 50  0001 C CNN
@@
 P 7450 3300
 AR Path="/5F315FB6/5FAAEDE1" Ref="R?"  Part="1"
-AR Path="/5FA4220C/5FAAEDE1" Ref="R66"  Part="1"
-F 0 "R66" H 7520 3346 50  0000 L CNN
+AR Path="/5FA4220C/5FAAEDE1" Ref="R59"  Part="1"
+F 0 "R59" H 7520 3346 50  0000 L CNN
 F 1 "1k" H 7520 3255 50  0000 L CNN
 F 2 "Resistor_SMD:R_0402_1005Metric" V 7380 3300 50  0001 C CNN
