File: obc_board/cubesat_obc 3.kicad_pcb (KiCad board)
At the start: 2 copper layers, 92 x 88.9 mm, 243 parts, among them J1 Conn_01x04_Female, J10 Conn_01x02_Female, J11 Conn_01x02_Female, J12 Conn_01x02_Female, J13 Conn_01x02_Female, J14 FSI-110-03-X-D-AD-SD-K-TR, J15 FSI-110-03-X-D-AD-SD-K-TR, J16 Conn_01x04_Female, J2 Conn_01x04_Female, J3 Conn_01x04_Female, J4 Conn_01x04_Female, J5 Conn_01x05_Female, J6 Conn_01x04_Female, J7 Conn_01x04_Female, J8 Conn_01x08_Female, J9 Micro_SD_Card, U1 AT45DB041E-SSHN-B, U10 BMM150, U11 LTC4304CMSTRPBF, U12 LTC4304CMSTRPBF, U13 PC104, U14 MAX14830, U15 AP2127N-3.3, U16 FT4232H-56Q-REEL, U2 AT45DB041E-SSHN-B, U3 STM32L552ZE, U4 LTC4304CMSTRPBF, U5 MCP9600-E_MX, U6 MCP9600-E_MX, U7 MCP9600-E_MX, U8 MCP9600-E_MX, U9 BMI160, Y1 32.768kHz, Y2 8MHz, Y3 4MHz, Y4 12MHz

Commit message: layout
Parts:
- removed C44, C47, C49, C50, C51, C52, C53, C54, C55: 100n, Capacitor_SMD:C_0402_1005Metric
- removed C45, C46: 20p, Capacitor_SMD:C_0201_0603Metric
- removed C48: 1u, Capacitor_SMD:C_0603_1608Metric
- removed J16: Conn_01x04_Female, Connector_Molex:Molex_PicoBlade_53261-0471_1x04-1MP_P1.25mm_Horizontal
- removed L9: 300n, Inductor_SMD:L_1210_3225Metric
- removed R111: 1k, Resistor_SMD:R_0402_1005Metric
- removed R112: 100k, Resistor_SMD:R_0402_1005Metric
- removed R113: 12k, Resistor_SMD:R_0201_0603Metric
- removed U15: AP2127N-3.3, Package_TO_SOT_SMD:SOT-23
- removed U16: FT4232H-56Q-REEL, cubesat_obc:QFN50P800X800X100-57N
- removed Y4: 12MHz, Crystal:Crystal_SMD_5032-4Pin_5.0x3.2mm
- moved R18 25.9 mm to (146.4, 106.8), turned to 270 degrees
- moved R19 24.6 mm to (144.8, 106.8), turned to 270 degrees
- moved R97 23.9 mm to (160.1, 64.3), turned to 90 degrees
- moved R98 21.3 mm to (162.4, 64.3), turned to 90 degrees
- moved R13 19.8 mm to (122.5, 103.7)
- moved R15 19.8 mm to (122.6, 107.3)
- moved R17 19.8 mm to (122.6, 110.9)
- moved R12 19.8 mm to (121.0, 103.7)
- moved R14 19.8 mm to (121.0, 107.3)
- moved R16 19.8 mm to (121.0, 110.9)
- moved R52 8.46 mm to (169.8, 95.6), turned to 180 degrees
- moved R56 6.65 mm to (169.8, 93.9), turned to 180 degrees
- moved FL2 6.41 mm to (129.5, 65.8)
- moved FL1 6.25 mm to (130.0, 109.0)
- moved R54 5.74 mm to (169.8, 92.3), turned to 180 degrees
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Connections:
- J14 pad 17: /TX0 -> /TX4
- J14 pad 18: /TX3 -> /TX1
- J14 pad 19: /RX0 -> /RX4
- J14 pad 20: /RX3 -> /RX1
- J15 pad 17: /TX1 -> /TX2
- J15 pad 18: /modules/UART3_RX -> /TX3
- J15 pad 19: /RX1 -> /RX2
- J15 pad 20: /modules/UART3_TX -> /RX3
- R12 pad 2: /mcu/USART3_TX -> /TX3
- R13 pad 2: /mcu/USART3_RX -> /RX3
- R14 pad 2: /mcu/USART2_TX -> /TX2
- R15 pad 2: /mcu/USART2_RX -> /RX2
- R16 pad 2: /mcu/USART1_TX -> /TX1
- R17 pad 2: /mcu/USART1_RX -> /RX1
- U3 pad 136: /mcu/USART1_TX -> /TX1
- U3 pad 137: /mcu/USART1_RX -> /RX1
- U3 pad 34: /RX2 -> /TX4
- U3 pad 35: /TX2 -> /RX4
- U3 pad 36: /mcu/USART2_TX -> /TX2
- U3 pad 37: /mcu/USART2_RX -> /RX2
- U3 pad 44: /mcu/USART3_TX -> /TX3
- U3 pad 45: /mcu/USART3_RX -> /RX3
Routing:
- net /MOSI_2: track 168.3 -> 0.00 mm, vias 3 -> 0
- net /SCK_2: track 157.1 -> 4.52 mm, vias 10 -> 2
- net /3V3_3: track 208.8 -> 86.1 mm, vias 37 -> 18
- net GND: track 293.9 -> 194.2 mm, vias 29 -> 15
- net /mcu/JTMS: track 81.0 -> 0.00 mm, vias 6 -> 0
- net /mcu/NRST: track 74.9 -> 0.00 mm, vias 6 -> 0
- net /SCL3: track 74.8 -> 0.00 mm, vias 5 -> 0
- net /CS3: track 70.7 -> 0.00 mm, vias 1 -> 0
- net /CS1: track 70.4 -> 0.00 mm, vias 2 -> 0
- net /SDA3: track 70.2 -> 0.00 mm, vias 5 -> 0
- net /VCC: track 69.0 -> 0.00 mm, vias 4 -> 0
- net /CS2: track 67.2 -> 0.00 mm, vias 2 -> 0
- net /mcu/NJRST: track 63.9 -> 0.00 mm, vias 2 -> 0
- net /3V3_2: track 67.5 -> 7.37 mm, vias 11 -> 0
- net /mcu/JTDO: track 59.8 -> 0.00 mm, vias 2 -> 0
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
Commit message: relayout
Parts:
- removed C11, C12, C14, C15, C3, C4, C5, C8: 100n, Capacitor_SMD:C_0402_1005Metric
- removed the C19 at (195.6, 83.9)
- removed the C20 at (195.5, 93.3)
- removed the C21 at (154.0, 92.4)
- removed the C22 at (153.8, 77.9)
- removed the C23 at (145.3, 99.3)
- removed the C24 at (153.9, 98.8)
- removed the C25 at (118.8, 54.8)
- removed the R11 at (164.0, 118.0)
- removed the R12 at (121.0, 103.7)
- removed the R13 at (122.5, 103.7)
- removed the R14 at (121.0, 107.3)
- removed the R15 at (122.6, 107.3)
- removed the R16 at (121.0, 110.9)
- removed the R17 at (122.6, 110.9)
- removed the R97 at (160.1, 64.3)
- removed the R98 at (162.4, 64.3)
- removed the U3 at (145.0, 90.4)
- added C39: 100n, Capacitor_SMD:C_0402_1005Metric, F.Cu at (188.7, 122.2)
- added C40: 20p, Capacitor_SMD:C_0201_0603Metric, B.Cu at (169.2, 118.4)
- added C41: 20p, Capacitor_SMD:C_0201_0603Metric, B.Cu at (169.2, 114.8)
- added C42: 100n, Capacitor_SMD:C_0402_1005Metric, F.Cu at (190.2, 124.5)
- added C43: 1u, Capacitor_SMD:C_0603_1608Metric, B.Cu at (181.6, 123.7)
- added C44: 100n, Capacitor_SMD:C_0402_1005Metric, B.Cu at (190.5, 114.3)
- added C45: 100n, Capacitor_SMD:C_0402_1005Metric, B.Cu at (184.4, 122.9)
- added C46: 100n, Capacitor_SMD:C_0402_1005Metric, B.Cu at (181.9, 125.2)
- added C47: 100n, Capacitor_SMD:C_0402_1005Metric, B.Cu at (189.5, 117.3)
- added C48: 100n, Capacitor_SMD:C_0402_1005Metric, B.Cu at (186.9, 122.9)
- added C49: 100n, Capacitor_SMD:C_0402_1005Metric, B.Cu at (182.4, 110.5)
- added C50: 100n, Capacitor_SMD:C_0402_1005Metric, B.Cu at (178.1, 119.4)
- added C51: 1u, Capacitor_SMD:C_0603_1608Metric, B.Cu at (130.8, 104.9)
- added C52: 100n, Capacitor_SMD:C_0402_1005Metric, B.Cu at (149.6, 114.3)
- added C53: 4.7u, Capacitor_SMD:C_0805_2012Metric, B.Cu at (133.1, 104.9)
- added C54: 100n, Capacitor_SMD:C_0402_1005Metric, B.Cu at (157.2, 89.4)
- added C55: 4.7u, Capacitor_SMD:C_0805_2012Metric, B.Cu at (157.0, 86.6)
- added C57: 100n, Capacitor_SMD:C_0402_1005Metric, B.Cu at (145.2, 89.4)
- added C58: 100n, Capacitor_SMD:C_0402_1005Metric, F.Cu at (140.0, 94.7)
- added C60: 100n, Capacitor_SMD:C_0402_1005Metric, B.Cu at (136.1, 111.5)
- added C62: 100n, Capacitor_SMD:C_0402_1005Metric, B.Cu at (150.7, 89.4)
- added C64: 100n, Capacitor_SMD:C_0402_1005Metric, B.Cu at (161.0, 98.8)
- added C66: 100n, Capacitor_SMD:C_0402_1005Metric, B.Cu at (161.0, 103.4)
- added C67: 100n, Capacitor_SMD:C_0402_1005Metric, B.Cu at (136.1, 105.0)
- added C68: 100n, Capacitor_SMD:C_0402_1005Metric, B.Cu at (136.4, 91.3)
- added C69: 100n, Capacitor_SMD:C_0402_1005Metric, B.Cu at (136.1, 99.7)
- added C71: 100n, Capacitor_SMD:C_0402_1005Metric, B.Cu at (155.3, 89.4)
- added C73: 100n, Capacitor_SMD:C_0402_1005Metric, B.Cu at (161.0, 110.1)
- added C74: 4.7u, Capacitor_SMD:C_0201_0603Metric, B.Cu at (135.1, 87.4)
- added J1: Conn_01x08_Female, Connector_Molex:Molex_PicoBlade_53261-0871_1x08-1MP_P1.25mm_Horizontal, B.Cu at (196.3, 121.4)
- added J15: Conn_01x04_Female, Connector_Molex:Molex_PicoBlade_53261-0471_1x04-1MP_P1.25mm_Horizontal, F.Cu at (196.3, 124.2)
- added L10: 4.7u, cubesat_obc:L_Vishay_IHLP-2020, B.Cu at (132.6, 93.2)
- added L9: 300n, Inductor_SMD:L_1210_3225Metric, B.Cu at (179.6, 128.8)
- added R112: 1k, Resistor_SMD:R_0402_1005Metric, B.Cu at (175.8, 114.0)
- added R113: 100k, Resistor_SMD:R_0402_1005Metric, B.Cu at (177.0, 113.3)
- added R114: 12k, Resistor_SMD:R_0201_0603Metric, B.Cu at (178.3, 116.8)
- added R21: 10k, Resistor_SMD:R_0402_1005Metric, B.Cu at (161.8, 100.6)
- added R24: 10k, Resistor_SMD:R_0402_1005Metric, B.Cu at (161.8, 101.7)
- added R62: 10k, Resistor_SMD:R_0402_1005Metric, F.Cu at (139.2, 110.2)
- added R63: 1k, Resistor_SMD:R_0402_1005Metric, F.Cu at (139.2, 112.5)
- added R64: 10k, Resistor_SMD:R_0402_1005Metric, F.Cu at (139.2, 108.0)
- added R65: 10k, Resistor_SMD:R_0402_1005Metric, F.Cu at (139.2, 105.7)
- added R66: 1k, Resistor_SMD:R_0402_1005Metric, F.Cu at (150.4, 106.2)
- added R67: 10k, Resistor_SMD:R_0402_1005Metric, F.Cu at (150.4, 108.7)
- added R68: 10k, Resistor_SMD:R_0402_1005Metric, F.Cu at (150.4, 111.0)
- added R69: 10k, Resistor_SMD:R_0402_1005Metric, F.Cu at (139.2, 87.6)
- added R70: 1k, Resistor_SMD:R_0402_1005Metric, F.Cu at (139.2, 89.9)
- added R71: 10k, Resistor_SMD:R_0402_1005Metric, F.Cu at (139.2, 85.3)
- added R72: 10k, Resistor_SMD:R_0402_1005Metric, F.Cu at (139.2, 83.1)
- added R73: 1k, Resistor_SMD:R_0402_1005Metric, F.Cu at (150.4, 83.8)
- added R74: 10k, Resistor_SMD:R_0402_1005Metric, F.Cu at (150.4, 86.4)
- added R75: 10k, Resistor_SMD:R_0402_1005Metric, F.Cu at (150.4, 88.6)
- added U13: LTC4304CMSTRPBF, Package_SO:MSOP-10_3x3mm_P0.5mm, F.Cu at (143.8, 109.5)
- added U15: LTC4304CMSTRPBF, Package_SO:MSOP-10_3x3mm_P0.5mm, F.Cu at (143.8, 86.9)
- added U17: AP2127N-3.3, Package_TO_SOT_SMD:SOT-23, F.Cu at (186.7, 125.5)
- added U18: FT4232H-56Q-REEL, cubesat_obc:QFN50P800X800X100-57N, B.Cu at (184.2, 116.1)
- added U19: STM32L552ZET6Q, Package_QFP:LQFP-144_20x20mm_P0.5mm, B.Cu at (148.6, 101.9)
- added Y2: 12MHz, Crystal:Crystal_SMD_5032-4Pin_5.0x3.2mm, B.Cu at (172.2, 116.6)
- C33: renamed from C34; footprint Capacitor_SMD:CP_Elec_4x5.3 -> Capacitor_SMD:C_1206_3216Metric; moved to B.Cu
- C34: renamed from C35; footprint Capacitor_SMD:CP_Elec_4x5.3 -> Capacitor_SMD:C_1206_3216Metric; moved to B.Cu
- C63: renamed from C17; moved to B.Cu
- C65: renamed from C18; footprint Capacitor_SMD:CP_Elec_4x5.3 -> Capacitor_SMD:C_0603_1608Metric
- R117: renamed from R20; moved to B.Cu
- R118: renamed from R21; moved to B.Cu
- R12: renamed from R96; moved to F.Cu
- R26: renamed from R35; moved to F.Cu
- R27: renamed from R36; moved to F.Cu
- R9: renamed from R95; moved to F.Cu
- U4: moved to F.Cu
- moved R119 88.6 mm to (151.0, 31.4)
- moved R120 88.6 mm to (148.1, 31.4)
- moved C34 77.2 mm to (122.4, 74.2), turned to 90 degrees
- moved C33 74.9 mm to (121.9, 119.9), turned to 90 degrees
- moved R3 54.3 mm to (142.5, 72.9), turned to 180 degrees
- moved R4 53.8 mm to (151.4, 72.9), turned to 0 degrees
- moved C19 51.4 mm to (142.5, 74.4), turned to 0 degrees
- moved C20 50.8 mm to (151.4, 74.4), turned to 0 degrees
- moved U2 41.1 mm to (142.6, 79.6), turned to 90 degrees
- moved U3 40.1 mm to (151.4, 79.8), turned to 90 degrees
- moved R7 34.0 mm to (139.2, 84.8), turned to 90 degrees
- moved R5 31.6 mm to (142.0, 84.8), turned to 90 degrees
- moved R6 29.5 mm to (150.6, 85.1), turned to 90 degrees
- moved R8 29.0 mm to (148.2, 85.1), turned to 90 degrees
- moved R115 25.9 mm to (120.8, 110.6), turned to 0 degrees
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- renumbered C1 to C19, C2 to C20, C26 to C21, C27 to C22, C36 to C23, C37 to C24, C28 to C25, C29 to C26, C38 to C27, C39 to C28, C30 to C29, C31 to C30, C32 to C31, C33 to C32, C40 to C35, C41 to C36, C42 to C37, C43 to C38, C9 to C56, C10 to C59, C16 to C61, C7 to C70, C6 to C72, C13 to C75, J15 to J10, J1 to J11, J2 to J12, J3 to J13, J4 to J14, J8 to J16, J9 to J17, J5 to J2, J6 to J3, J7 to J4, J10 to J5, J11 to J6, J12 to J7, J13 to J8, J14 to J9, R22 to R10, R99 to R100, R100 to R101, R101 to R102, R102 to R103, R103 to R104, R104 to R105, R105 to R106, R106 to R107, R107 to R108, R108 to R109, R23 to R11, R109 to R110, R110 to R111, R18 to R115, R19 to R116, R9 to R119, R10 to R120, R24 to R13, R25 to R14, R26 to R15, R27 to R16, R28 to R17, R29 to R18, R30 to R19, R31 to R20, R32 to R22, R33 to R23, R34 to R25, R37 to R28, R38 to R29, R39 to R30, R40 to R31, R41 to R32, R42 to R33, R43 to R34, R44 to R35, R45 to R36, R46 to R37, R47 to R38, R48 to R39, R49 to R40, R50 to R41, R51 to R42, R52 to R43, R53 to R44, R54 to R45, R55 to R46, R56 to R47, R57 to R48, R58 to R49, R59 to R50, R60 to R51, R61 to R52, R62 to R53, R63 to R54, R64 to R55, R65 to R56, R66 to R57, R67 to R58, R68 to R59, R69 to R60, R70 to R61, R71 to R76, R72 to R77, R73 to R78, R74 to R79, R75 to R80, R76 to R81, R77 to R82, R78 to R83, R79 to R84, R80 to R85, R81 to R86, R82 to R87, R83 to R88, R84 to R89, R85 to R90, R86 to R91, R87 to R92, R88 to R93, R89 to R94, R90 to R95, R91 to R96, R92 to R97, R93 to R98, R94 to R99, U13 to U14, U14 to U16, U1 to U2, U2 to U3, Y3 to Y1, Y2 to Y3, Y1 to Y4
Connections:
- net /mcu/OSC_IN renamed Net-(C56-Pad1)
- net /mcu/OSC_OUT renamed Net-(C59-Pad1)
- J10 pad 17: /TX2 -> /RX3_OBC
- J10 pad 18: /TX3 -> /modules/UART3_RX
- J10 pad 19: /RX2 -> /TX3_OBC
- J10 pad 20: /RX3 -> /modules/UART3_TX
- J11 pad 1: /VCC -> GND
- J11 pad 2: /uart_expander/TX0 -> /VCC
- J11 pad 4: GND -> /uart_expander/TX0
- J12 pad 1: /VCC -> GND
- J12 pad 2: /uart_expander/TX1 -> /VCC
- J12 pad 4: GND -> /uart_expander/TX1
- J13 pad 1: /VCC -> GND
- J13 pad 2: /uart_expander/TX2 -> /VCC
- J13 pad 4: GND -> /uart_expander/TX2
- J14 pad 1: /VCC -> GND
- J14 pad 2: /uart_expander/TX3 -> /VCC
- J14 pad 4: GND -> /uart_expander/TX3
- J16 pad 1: /mcu/JTDI -> GND
- J16 pad 2: /mcu/JTDO -> /3V3_3
- J16 pad 3: /mcu/JTMS -> /mcu/JTDI
- J16 pad 4: /mcu/JTCK -> /mcu/JTDO
- J16 pad 5: /mcu/NRST -> /mcu/JTMS
- J16 pad 6: /mcu/NJRST -> /mcu/JTCK
- J16 pad 7: GND -> /mcu/NRST
- J16 pad 8: /3V3_3 -> /mcu/NJTRST
- J2 pad 1: /SCK_2 -> GND
- J2 pad 2: /MOSI_2 -> /SCK_2
- J2 pad 3: /MISO_2 -> /MOSI_2
- J2 pad 4: /CS3 -> /MISO_2
- J2 pad 5: GND -> /CS3
- J3 pad 1: /ADC1 -> GND
- J3 pad 2: /ADC2 -> /ADC1
- J3 pad 3: /ADC3 -> /ADC2
- J3 pad 4: GND -> /ADC3
- J4 pad 1: /ADC4 -> GND
- J4 pad 2: /ADC5 -> /ADC4
- J4 pad 3: /ADC6 -> /ADC5
- J4 pad 4: GND -> /ADC6
- J9 pad 17: /TX4 -> /TX1_OBC
- J9 pad 18: /TX1 -> /RX2_OBC
- J9 pad 19: /RX4 -> /RX1_OBC
- J9 pad 20: /RX1 -> /TX2_OBC
- R104 pad 2: /uart_expander/TX0 -> /uart_expander/RX0
- R105 pad 2: /uart_expander/TX1 -> /uart_expander/RX1
- R106 pad 2: /uart_expander/TX2 -> /uart_expander/RX2
- R107 pad 2: /uart_expander/TX3 -> /uart_expander/RX3
- R108 pad 2: /uart_expander/RX0 -> /uart_expander/TX0
- R109 pad 2: /uart_expander/RX1 -> /uart_expander/TX1
- R110 pad 2: /uart_expander/RX2 -> /uart_expander/TX2
- R111 pad 2: /uart_expander/RX3 -> /uart_expander/TX3
- R117 pad 1: /SDA3 -> /SDA4
- R118 pad 1: /SCL3 -> /SCL4
- U14 pad 11: /SDA2 -> Net-(R63-Pad2)
- U14 pad 41: /SCL3 -> Net-(R73-Pad1)
- U14 pad 43: /SDA3 -> Net-(R70-Pad2)
- U14 pad 53: /TX4 -> Net-(U14-Pad53)
- U14 pad 55: /RX4 -> Net-(U14-Pad55)
- U14 pad 57: /TX3 -> Net-(U14-Pad57)
- U14 pad 59: /RX3 -> Net-(U14-Pad59)
- U14 pad 9: /SCL2 -> Net-(R66-Pad1)
- U2 pad 1: /MISO_3 -> /MISO_1
- U2 pad 2: /SCK_3 -> /SCK_1
- U2 pad 8: /MOSI_3 -> /MOSI_1
- U3 pad 1: /MISO_3 -> /MISO_1
- U3 pad 2: /SCK_3 -> /SCK_1
- U3 pad 8: /MOSI_3 -> /MOSI_1
- U9 pad 1: /MISO_1 -> /MISO_2
- U9 pad 13: /SCK_1 -> /SCK_2
- U9 pad 14: /MOSI_1 -> /MOSI_2
Routing:
- net GND: track 194.2 -> 341.3 mm, vias 15 -> 9
- net /MOSI_2: track 0.00 -> 94.8 mm, vias 0 -> 4
- net /MISO_2: track 4.55 -> 90.3 mm, vias 2 -> 3
- net /SCK_2: track 4.52 -> 84.3 mm, vias 2 -> 1
- net /sensors/SDA: track 67.6 -> 0.00 mm, vias 7 -> 0
- net /sensors/SCL: track 60.4 -> 0.00 mm, vias 5 -> 0
- net /3V3_3: track 86.1 -> 143.0 mm, vias 18 -> 23
- net /MOSI_3: track 53.5 -> 0.00 mm
- net /mcu/NRST: track 0.00 -> 53.3 mm, vias 0 -> 2
- net /SCK_3: track 52.5 -> 0.00 mm
- net /mcu/JTMS: track 0.00 -> 50.9 mm, vias 0 -> 2
- net Net-(C74-Pad2): track 0.00 -> 50.8 mm, vias 0 -> 2
- net /MISO_3: track 46.3 -> 0.00 mm, vias 4 -> 0
- net (no net): track 0.00 -> 41.9 mm
- net /mcu/NJTRST: track 0.00 -> 39.1 mm, vias 0 -> 2
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