File: obc_board/sensors.sch (KiCad schematic (older format))
At the start: 86 parts, among them J10 Conn_01x02_Female, J11 Conn_01x02_Female, J12 Conn_01x02_Female, J13 Conn_01x02_Female, U10 BMM150, U4 LTC4304CMSTRPBF, U5 MCP9600-E_MX, U6 MCP9600-E_MX, U7 MCP9600-E_MX, U8 MCP9600-E_MX, U9 BMI160

Commit message: layout done
Parts:
- renumbered C36 to C28, C37 to C29, C28 to C30, C29 to C31, C38 to C32, C39 to C33, C30 to C34, C31 to C35, C32 to C36, C33 to C37, J10 to J6, J11 to J7, J12 to J8, J13 to J9, R95 to R16, R22 to R17, R23 to R18, R96 to R19, R24 to R20, R25 to R21, R26 to R22, R27 to R23, R28 to R24, R29 to R25, R30 to R26, R31 to R27, R97 to R28, R32 to R29, R33 to R30, R98 to R31, R34 to R32, R35 to R33, R36 to R34, R37 to R35, R38 to R36, R39 to R37, R40 to R38, R41 to R39, R42 to R40, R43 to R41, R44 to R42, R45 to R43, R46 to R44, R47 to R45, R48 to R46, R49 to R47, R50 to R48, R51 to R49, R52 to R50, R53 to R51, R54 to R52, R55 to R53, R56 to R54

Commit message: relayout
Parts:
- removed R28, R31: 10k, Resistor_SMD:R_0402_1005Metric, symbol Device:R
- renumbered C26 to C21, C27 to C22, C28 to C23, C29 to C24, C30 to C25, C31 to C26, C32 to C27, C33 to C28, C34 to C29, C35 to C30, C36 to C31, C37 to C32, J6 to J5, J7 to J6, J8 to J7, J9 to J8, R17 to R10, R18 to R11, R19 to R12, R20 to R13, R21 to R14, R22 to R15, R23 to R16, R24 to R17, R25 to R18, R26 to R19, R27 to R20, R29 to R22, R30 to R23, R32 to R25, R33 to R26, R34 to R27, R35 to R28, R36 to R29, R37 to R30, R38 to R31, R39 to R32, R40 to R33, R41 to R34, R42 to R35, R43 to R36, R44 to R37, R45 to R38, R46 to R39, R47 to R40, R48 to R41, R49 to R42, R50 to R43, R51 to R44, R52 to R45, R53 to R46, R54 to R47, R16 to R9
Other:
- moved on the sheet: R12, R9
