File: obc_board/stacking_connector.sch (KiCad schematic (older format))
At the start: 25 parts

Commit message: pcb layout
Parts:
- R71, R72, R73, R74, R75, R76, R77, R78, R79, R80, R81, R82, R83, R84, R85, R86, R87, R88, R89, R90, R91, R92, R93, R94: renamed from R?; footprint (none) -> Resistor_SMD:R_0402_1005Metric; Digikey Part Number (none) -> 311-0.0JRTR-ND
- gave numbers to parts that had none: 1
Connections:
- net 3V3_4 renamed VCC

Commit message: layout done
Parts:
- renumbered R71 to R69, R72 to R70, R73 to R71, R74 to R72, R75 to R73, R76 to R74, R77 to R75, R78 to R76, R79 to R77, R80 to R78, R81 to R79, R82 to R80, R83 to R81, R84 to R82, R85 to R83, R86 to R84, R87 to R85, R88 to R86, R89 to R87, R90 to R88, R91 to R89, R92 to R90, R93 to R91, R94 to R92
Connections:
- net RX1: no longer names the net of U13.55 (03)
- net RX2: no longer names the net of U13.59 (07)
- net TX1: no longer names the net of U13.53 (01)
- net TX2: no longer names the net of U13.57 (05)
Changed lines of the file:
@@
 OUT6
 $Comp
-L Device:R R71
+L Device:R R69
 U 1 1 5F471BF1
 P 7600 2300
-F 0 "R71" H 7670 2346 50  0000 L CNN
+F 0 "R69" H 7670 2346 50  0000 L CNN
 F 1 "0" H 7670 2255 50  0000 L CNN
 F 2 "Resistor_SMD:R_0402_1005Metric" V 7530 2300 50  0001 C CNN
@@
 $EndComp
 $Comp
-L Device:R R73
+L Device:R R71
 U 1 1 5F471FDD
 P 7850 2300
-F 0 "R73" H 7920 2346 50  0000 L CNN
+F 0 "R71" H 7920 2346 50  0000 L CNN
 F 1 "0" H 7920 2255 50  0000 L CNN
 F 2 "Resistor_SMD:R_0402_1005Metric" V 7780 2300 50  0001 C CNN
@@
 $EndComp
 $Comp
-L Device:R R75
+L Device:R R73
 U 1 1 5F4722B8
 P 8100 2300
-F 0 "R75" H 8170 2346 50  0000 L CNN
+F 0 "R73" H 8170 2346 50  0000 L CNN
 F 1 "0" H 8170 2255 50  0000 L CNN
 F 2 "Resistor_SMD:R_0402_1005Metric" V 8030 2300 50  0001 C CNN
@@
 $EndComp
 $Comp
-L Device:R R77
+L Device:R R75
 U 1 1 5F472497
 P 8350 2300
-F 0 "R77" H 8420 2346 50  0000 L CNN
+F 0 "R75" H 8420 2346 50  0000 L CNN
 F 1 "0" H 8420 2255 50  0000 L CNN
 F 2 "Resistor_SMD:R_0402_1005Metric" V 8280 2300 50  0001 C CNN
@@
 $EndComp
 $Comp
-L Device:R R79
+L Device:R R77
 U 1 1 5F472AE3
 P 8600 2300
-F 0 "R79" H 8670 2346 50  0000 L CNN
+F 0 "R77" H 8670 2346 50  0000 L CNN
 F 1 "0" H 8670 2255 50  0000 L CNN
 F 2 "Resistor_SMD:R_0402_1005Metric" V 8530 2300 50  0001 C CNN
@@
 $EndComp
 $Comp
-L Device:R R81
+L Device:R R79
 U 1 1 5F472C83
 P 8850 2300
-F 0 "R81" H 8920 2346 50  0000 L CNN
+F 0 "R79" H 8920 2346 50  0000 L CNN
 F 1 "0" H 8920 2255 50  0000 L CNN
 F 2 "Resistor_SMD:R_0402_1005Metric" V 8780 2300 50  0001 C CNN
@@
 	9200 3350 9600 3350
 $Comp
-L Device:R R83
+L Device:R R81
 U 1 1 5F495AD2
 P 9600 2300
-F 0 "R83" H 9670 2346 50  0000 L CNN
+F 0 "R81" H 9670 2346 50  0000 L CNN
 F 1 "0" H 9670 2255 50  0000 L CNN
 F 2 "Resistor_SMD:R_0402_1005Metric" V 9530 2300 50  0001 C CNN
@@
 $EndComp
 $Comp
-L Device:R R85
+L Device:R R83
 U 1 1 5F495AD8
 P 9850 2300
-F 0 "R85" H 9920 2346 50  0000 L CNN
+F 0 "R83" H 9920 2346 50  0000 L CNN
 F 1 "0" H 9920 2255 50  0000 L CNN
 F 2 "Resistor_SMD:R_0402_1005Metric" V 9780 2300 50  0001 C CNN
@@
 $EndComp
 $Comp
-L Device:R R87
+L Device:R R85
 U 1 1 5F495ADE
 P 10100 2300
-F 0 "R87" H 10170 2346 50  0000 L CNN
+F 0 "R85" H 10170 2346 50  0000 L CNN
 F 1 "0" H 10170 2255 50  0000 L CNN
 F 2 "Resistor_SMD:R_0402_1005Metric" V 10030 2300 50  0001 C CNN
@@
 $EndComp
 $Comp
-L Device:R R89
+L Device:R R87
 U 1 1 5F495AE4
 P 10350 2300
-F 0 "R89" H 10420 2346 50  0000 L CNN
+F 0 "R87" H 10420 2346 50  0000 L CNN
 F 1 "0" H 10420 2255 50  0000 L CNN
 F 2 "Resistor_SMD:R_0402_1005Metric" V 10280 2300 50  0001 C CNN
@@
 $EndComp
 $Comp
-L Device:R R91
+L Device:R R89
 U 1 1 5F495AEA
 P 10600 2300
-F 0 "R91" H 10670 2346 50  0000 L CNN
+F 0 "R89" H 10670 2346 50  0000 L CNN
 F 1 "0" H 10670 2255 50  0000 L CNN
 F 2 "Resistor_SMD:R_0402_1005Metric" V 10530 2300 50  0001 C CNN
@@
 $EndComp
 $Comp
-L Device:R R93
+L Device:R R91
 U 1 1 5F495AF0
 P 10850 2300
-F 0 "R93" H 10920 2346 50  0000 L CNN
+F 0 "R91" H 10920 2346 50  0000 L CNN
 F 1 "0" H 10920 2255 50  0000 L CNN
 F 2 "Resistor_SMD:R_0402_1005Metric" V 10780 2300 50  0001 C CNN
@@
 $EndComp
 $Comp
-L Device:R R84
+L Device:R R82
 U 1 1 5F499B14
 P 9600 3700
-F 0 "R84" H 9670 3746 50  0000 L CNN
+F 0 "R82" H 9670 3746 50  0000 L CNN
 F 1 "0" H 9670 3655 50  0000 L CNN
 F 2 "Resistor_SMD:R_0402_1005Metric" V 9530 3700 50  0001 C CNN
@@
 $EndComp
 $Comp
-L Device:R R86
+L Device:R R84
 U 1 1 5F499B1A
 P 9850 3700
-F 0 "R86" H 9920 3746 50  0000 L CNN
+F 0 "R84" H 9920 3746 50  0000 L CNN
 F 1 "0" H 9920 3655 50  0000 L CNN
 F 2 "Resistor_SMD:R_0402_1005Metric" V 9780 3700 50  0001 C CNN
@@
 $EndComp
 $Comp
-L Device:R R88
+L Device:R R86
 U 1 1 5F499B20
 P 10100 3700
-F 0 "R88" H 10170 3746 50  0000 L CNN
+F 0 "R86" H 10170 3746 50  0000 L CNN
 F 1 "0" H 10170 3655 50  0000 L CNN
 F 2 "Resistor_SMD:R_0402_1005Metric" V 10030 3700 50  0001 C CNN
@@
 $EndComp
 $Comp
-L Device:R R90
+L Device:R R88
 U 1 1 5F499B26
 P 10350 3700
-F 0 "R90" H 10420 3746 50  0000 L CNN
+F 0 "R88" H 10420 3746 50  0000 L CNN
 F 1 "0" H 10420 3655 50  0000 L CNN
 F 2 "Resistor_SMD:R_0402_1005Metric" V 10280 3700 50  0001 C CNN
@@
 $EndComp
 $Comp
-L Device:R R92
+L Device:R R90
 U 1 1 5F499B2C
 P 10600 3700
-F 0 "R92" H 10670 3746 50  0000 L CNN
+F 0 "R90" H 10670 3746 50  0000 L CNN
 F 1 "0" H 10670 3655 50  0000 L CNN
 F 2 "Resistor_SMD:R_0402_1005Metric" V 10530 3700 50  0001 C CNN
@@
 $EndComp
 $Comp
-L Device:R R94
+L Device:R R92
 U 1 1 5F499B32
 P 10850 3700
-F 0 "R94" H 10920 3746 50  0000 L CNN
+F 0 "R92" H 10920 3746 50  0000 L CNN
 F 1 "0" H 10920 3655 50  0000 L CNN
 F 2 "Resistor_SMD:R_0402_1005Metric" V 10780 3700 50  0001 C CNN
@@
 $EndComp
 $Comp
-L Device:R R72
+L Device:R R70
 U 1 1 5F49D2BA
 P 7600 3700
-F 0 "R72" H 7670 3746 50  0000 L CNN
+F 0 "R70" H 7670 3746 50  0000 L CNN
 F 1 "0" H 7670 3655 50  0000 L CNN
 F 2 "Resistor_SMD:R_0402_1005Metric" V 7530 3700 50  0001 C CNN
@@
 $EndComp
 $Comp
-L Device:R R74
+L Device:R R72
 U 1 1 5F49D2C0
 P 7850 3700
-F 0 "R74" H 7920 3746 50  0000 L CNN
+F 0 "R72" H 7920 3746 50  0000 L CNN
 F 1 "0" H 7920 3655 50  0000 L CNN
 F 2 "Resistor_SMD:R_0402_1005Metric" V 7780 3700 50  0001 C CNN
@@
 $EndComp
 $Comp
-L Device:R R76
+L Device:R R74
 U 1 1 5F49D2C6
 P 8100 3700
-F 0 "R76" H 8170 3746 50  0000 L CNN
+F 0 "R74" H 8170 3746 50  0000 L CNN
 F 1 "0" H 8170 3655 50  0000 L CNN
 F 2 "Resistor_SMD:R_0402_1005Metric" V 8030 3700 50  0001 C CNN
@@
 $EndComp
 $Comp
-L Device:R R78
+L Device:R R76
 U 1 1 5F49D2CC
 P 8350 3700
-F 0 "R78" H 8420 3746 50  0000 L CNN
+F 0 "R76" H 8420 3746 50  0000 L CNN
 F 1 "0" H 8420 3655 50  0000 L CNN
 F 2 "Resistor_SMD:R_0402_1005Metric" V 8280 3700 50  0001 C CNN
@@
 $EndComp
 $Comp
-L Device:R R80
+L Device:R R78
 U 1 1 5F49D2D2
 P 8600 3700
-F 0 "R80" H 8670 3746 50  0000 L CNN
+F 0 "R78" H 8670 3746 50  0000 L CNN
 F 1 "0" H 8670 3655 50  0000 L CNN
 F 2 "Resistor_SMD:R_0402_1005Metric" V 8530 3700 50  0001 C CNN
@@
 $EndComp
 $Comp
-L Device:R R82
+L Device:R R80
 U 1 1 5F49D2D8
 P 8850 3700
-F 0 "R82" H 8920 3746 50  0000 L CNN
+F 0 "R80" H 8920 3746 50  0000 L CNN
 F 1 "0" H 8920 3655 50  0000 L CNN
 F 2 "Resistor_SMD:R_0402_1005Metric" V 8780 3700 50  0001 C CNN
@@
 Text HLabel 5400 2300 2    50   Input ~ 0
 CS2
-Text HLabel 3850 1900 0    50   Input ~ 0
-TX1
-Text HLabel 3850 2000 0    50   Input ~ 0
-RX1
-Text HLabel 3850 2100 0    50   Input ~ 0
-TX2
-Text HLabel 3850 2200 0    50   Input ~ 0
-RX2
 Text HLabel 1400 4000 0    50   Input ~ 0
 SCL1

Commit message: relayout
Parts:
- added R62, R64, R65, R67, R68, R69, R71, R72, R74, R75: 10k, Resistor_SMD:R_0402_1005Metric, symbol Device:R
- added R63, R66, R70, R73: 1k, Resistor_SMD:R_0402_1005Metric, symbol Device:R
- added U13, U15: LTC4304CMSTRPBF, Package_SO:MSOP-10_3x3mm_P0.5mm, symbol cubesat_obc_lib:LTC4304CMSTRPBF
- renumbered R69 to R76, R70 to R77, R71 to R78, R72 to R79, R73 to R80, R74 to R81, R75 to R82, R76 to R83, R77 to R84, R78 to R85, R79 to R86, R80 to R87, R81 to R88, R82 to R89, R83 to R90, R84 to R91, R85 to R92, R86 to R93, R87 to R94, R88 to R95, R89 to R96, R90 to R97, R91 to R98, R92 to R99, U13 to U14
Connections:
- net 3V3_3: now also R62.1, R64.1, R65.1, R67.1, R68.1, R69.1, R71.1, R72.1, R74.1, R75.1, U13.10 (VCC), U15.10 (VCC)
- net GND: now also U13.5 (GND), U15.5 (GND)
- net SCL1: now also U13.3 (SCLIN); no longer U14.43 (43-I2C-SCL)
- net SCL2: now also U15.3 (SCLIN); no longer U14.11 (11-I2C2_SCL)
- net SDA1: now also U13.8 (SDAIN); no longer U14.41 (41-I2C-SDA)
- net SDA2: now also U15.8 (SDAIN); no longer U14.9 (09-I2C2_SDA)
- new net: R65.2, U13.1 (ENABLE)
- new net: R63.1, R64.2, U13.2 (SCLOUT)
- new net: R66.2, R67.2, U13.9 (SDAOUT)
- new net: R63.2, U14.11 (11-I2C2_SCL)
- new net: R66.1, U14.9 (09-I2C2_SDA)
- new net: R73.1, U14.41 (41-I2C-SDA)
- new net: R70.2, U14.43 (43-I2C-SCL)
- new net: R72.2, U15.1 (ENABLE)
- new net: R70.1, R71.2, U15.2 (SCLOUT)
- new net: R73.2, R74.2, U15.9 (SDAOUT)
- new net ACC3: R62.2, U13.4 (*ACC)
- new net ACC4: R69.2, U15.4 (*ACC)
- new net FAULT3: R68.2, U13.7 (*FAULT)
- new net FAULT4: R75.2, U15.7 (*FAULT)
Other:
- moved on the sheet: U14
