File: obc_board/uart_expander.sch (KiCad schematic (older format))
At the start: 1 part

Commit message: layout
Parts:
- added C40, C41, C42, C43: 100n, Capacitor_SMD:C_0402_1005Metric, symbol Device:C
- added J1, J2, J3, J4: Conn_01x04_Female, Connector_Molex:Molex_PicoBlade_53261-0471_1x04-1MP_P1.25mm_Horizontal, symbol Connector:Conn_01x04_Female
- added R100, R101, R102, R99: 10k, Resistor_SMD:R_0402_1005Metric, symbol Device:R
- added R103, R104, R105, R106, R107, R108, R109, R110: 100k, Resistor_SMD:R_0402_1005Metric, symbol Device:R
- added Y3: 4MHz, Crystal:Crystal_SMD_MicroCrystal_CC1V-T1A-2Pin_8.0x3.7mm, symbol Device:Crystal
- U14: renamed from U?; Digikey Part Number (none) -> MAX14830ETM+-ND
Connections:
- net at U14.1 (SPI/~I2C): now also R102.2
- net GND: now reaches U14.10 (DGND)
- net GND: now also U14.46 (AGND), U14.49 (AGND), C40.2, C41.2, C42.2, C43.2, J1.4 (Pin_4), J2.4 (Pin_4), J3.4 (Pin_4), J4.4 (Pin_4)
- net RX0: now reaches U14.17 (RX0)
- net RX0: now also J1.3 (Pin_3), R107.2
- net TX0: now reaches U14.18 (TX0)
- net TX0: now also J1.2 (Pin_2), R103.2
- net 3V3: now reaches U14.2 (LDOEN)
- net 3V3: now also U14.43 (VEXT), U14.47 (VA), U14.9 (VL), C41.1, C42.1, C43.1, R100.1, R101.1, R102.1, R99.1
- net RX1: now reaches U14.25 (RX1)
- net RX1: now also J2.3 (Pin_3), R108.2
- net TX1: now reaches U14.26 (TX1)
- net TX1: now also J2.2 (Pin_2), R104.2
- net MISO: now reaches U14.3 (MISO/SDA)
- net RX2: now reaches U14.33 (RX2)
- net RX2: now also J3.3 (Pin_3), R109.2
- net TX2: now reaches U14.34 (TX2)
- net TX2: now also J3.2 (Pin_2), R105.2
- net SCK: now reaches U14.4 (SCLK/SCL)
- net RX3: now reaches U14.41 (RX3)
- net RX3: now also J4.3 (Pin_3), R110.2
- net TX3: now reaches U14.42 (TX3)
- net TX3: now also J4.2 (Pin_2), R106.2
- net at U14.44 (XOUT): now also Y3.1
- net at U14.45 (XIN): now also Y3.2
- net at U14.48 (V18): now also C40.1
- net CS: now reaches U14.5 (~CS~/A0)
- net CS: now also R101.2
- net MOSI: now reaches U14.6 (MOSI/A1)
- net IRQ: now reaches U14.7 (~IRQ)
- net IRQ: now also R99.2
- net RST: now reaches U14.8 (~RST)
- net RST: now also R100.2
- new net VCC: J1.1 (Pin_1), J2.1 (Pin_1), J3.1 (Pin_1), J4.1 (Pin_1), R103.1, R104.1, R105.1, R106.1, R107.1, R108.1, R109.1, R110.1

Commit message: layout done
Parts:
- renumbered J1 to J12, J2 to J13, J3 to J14, J4 to J15, R106 to R100, R107 to R101, R108 to R102, R109 to R103, R110 to R104, R99 to R93, R100 to R94, R101 to R95, R102 to R96, R103 to R97, R104 to R98, R105 to R99
Changed lines of the file:
@@
 3V3
 $Comp
-L Device:R R102
+L Device:R R96
 U 1 1 5F35B981
 P 3500 3500
-F 0 "R102" H 3570 3546 50  0000 L CNN
+F 0 "R96" H 3570 3546 50  0000 L CNN
 F 1 "10k" H 3570 3455 50  0000 L CNN
 F 2 "Resistor_SMD:R_0402_1005Metric" V 3430 3500 50  0001 C CNN
@@
 	2050 4350 2450 4350
 $Comp
-L Device:R R99
+L Device:R R93
 U 1 1 5F35E104
 P 2450 3650
-F 0 "R99" H 2520 3696 50  0000 L CNN
+F 0 "R93" H 2520 3696 50  0000 L CNN
 F 1 "10k" H 2520 3605 50  0000 L CNN
 F 2 "Resistor_SMD:R_0402_1005Metric" V 2380 3650 50  0001 C CNN
@@
 $EndComp
 $Comp
-L Device:R R100
+L Device:R R94
 U 1 1 5F35E5F6
 P 2750 3650
-F 0 "R100" H 2820 3696 50  0000 L CNN
+F 0 "R94" H 2820 3696 50  0000 L CNN
 F 1 "10k" H 2820 3605 50  0000 L CNN
 F 2 "Resistor_SMD:R_0402_1005Metric" V 2680 3650 50  0001 C CNN
@@
 	2750 4250 3900 4250
 $Comp
-L Device:R R101
+L Device:R R95
 U 1 1 5F360EEB
 P 3050 3650
-F 0 "R101" H 3120 3696 50  0000 L CNN
+F 0 "R95" H 3120 3696 50  0000 L CNN
 F 1 "10k" H 3120 3605 50  0000 L CNN
 F 2 "Resistor_SMD:R_0402_1005Metric" V 2980 3650 50  0001 C CNN
@@
 P 7750 3150
 AR Path="/5F37ABAA" Ref="J?"  Part="1"
-AR Path="/5F6EB2F1/5F37ABAA" Ref="J1"  Part="1"
-F 0 "J1" H 7778 3126 50  0000 L CNN
+AR Path="/5F6EB2F1/5F37ABAA" Ref="J12"  Part="1"
+F 0 "J12" H 7778 3126 50  0000 L CNN
 F 1 "Conn_01x04_Female" H 7778 3035 50  0000 L CNN
 F 2 "Connector_Molex:Molex_PicoBlade_53261-0471_1x04-1MP_P1.25mm_Horizontal" H 7750 3150 50  0001 C CNN
@@
 P 7750 3900
 AR Path="/5F37ABB1" Ref="J?"  Part="1"
-AR Path="/5F6EB2F1/5F37ABB1" Ref="J2"  Part="1"
-F 0 "J2" H 7778 3876 50  0000 L CNN
+AR Path="/5F6EB2F1/5F37ABB1" Ref="J13"  Part="1"
+F 0 "J13" H 7778 3876 50  0000 L CNN
 F 1 "Conn_01x04_Female" H 7778 3785 50  0000 L CNN
 F 2 "Connector_Molex:Molex_PicoBlade_53261-0471_1x04-1MP_P1.25mm_Horizontal" H 7750 3900 50  0001 C CNN
@@
 P 7750 4650
 AR Path="/5F37ABB8" Ref="J?"  Part="1"
-AR Path="/5F6EB2F1/5F37ABB8" Ref="J3"  Part="1"
-F 0 "J3" H 7778 4626 50  0000 L CNN
+AR Path="/5F6EB2F1/5F37ABB8" Ref="J14"  Part="1"
+F 0 "J14" H 7778 4626 50  0000 L CNN
 F 1 "Conn_01x04_Female" H 7778 4535 50  0000 L CNN
 F 2 "Connector_Molex:Molex_PicoBlade_53261-0471_1x04-1MP_P1.25mm_Horizontal" H 7750 4650 50  0001 C CNN
@@
 P 7750 5400
 AR Path="/5F37ABBF" Ref="J?"  Part="1"
-AR Path="/5F6EB2F1/5F37ABBF" Ref="J4"  Part="1"
-F 0 "J4" H 7778 5376 50  0000 L CNN
+AR Path="/5F6EB2F1/5F37ABBF" Ref="J15"  Part="1"
+F 0 "J15" H 7778 5376 50  0000 L CNN
 F 1 "Conn_01x04_Female" H 7778 5285 50  0000 L CNN
 F 2 "Connector_Molex:Molex_PicoBlade_53261-0471_1x04-1MP_P1.25mm_Horizontal" H 7750 5400 50  0001 C CNN
@@
 VCC
 $Comp
-L Device:R R103
+L Device:R R97
 U 1 1 5F38F396
 P 6800 2900
-F 0 "R103" H 6870 2946 50  0000 L CNN
+F 0 "R97" H 6870 2946 50  0000 L CNN
 F 1 "100k" H 6870 2855 50  0000 L CNN
 F 2 "Resistor_SMD:R_0402_1005Metric" V 6730 2900 50  0001 C CNN
@@
 	6800 3150 7550 3150
 $Comp
-L Device:R R107
+L Device:R R101
 U 1 1 5F393783
 P 7150 2900
-F 0 "R107" H 7220 2946 50  0000 L CNN
+F 0 "R101" H 7220 2946 50  0000 L CNN
 F 1 "100k" H 7220 2855 50  0000 L CNN
 F 2 "Resistor_SMD:R_0402_1005Metric" V 7080 2900 50  0001 C CNN
@@
 VCC
 $Comp
-L Device:R R104
+L Device:R R98
 U 1 1 5F39805E
 P 6800 3650
-F 0 "R104" H 6870 3696 50  0000 L CNN
+F 0 "R98" H 6870 3696 50  0000 L CNN
 F 1 "100k" H 6870 3605 50  0000 L CNN
 F 2 "Resistor_SMD:R_0402_1005Metric" V 6730 3650 50  0001 C CNN
@@
 	6800 3350 6800 3500
 $Comp
-L Device:R R108
+L Device:R R102
 U 1 1 5F398066
 P 7150 3650
-F 0 "R108" H 7220 3696 50  0000 L CNN
+F 0 "R102" H 7220 3696 50  0000 L CNN
 F 1 "100k" H 7220 3605 50  0000 L CNN
 F 2 "Resistor_SMD:R_0402_1005Metric" V 7080 3650 50  0001 C CNN
@@
 VCC
 $Comp
-L Device:R R105
+L Device:R R99
 U 1 1 5F39BCAA
 P 6800 4400
-F 0 "R105" H 6870 4446 50  0000 L CNN
+F 0 "R99" H 6870 4446 50  0000 L CNN
 F 1 "100k" H 6870 4355 50  0000 L CNN
 F 2 "Resistor_SMD:R_0402_1005Metric" V 6730 4400 50  0001 C CNN
@@
 	6800 4100 6800 4250
 $Comp
-L Device:R R109
+L Device:R R103
 U 1 1 5F39BCB2
 P 7150 4400
-F 0 "R109" H 7220 4446 50  0000 L CNN
+F 0 "R103" H 7220 4446 50  0000 L CNN
 F 1 "100k" H 7220 4355 50  0000 L CNN
 F 2 "Resistor_SMD:R_0402_1005Metric" V 7080 4400 50  0001 C CNN
@@
 VCC
 $Comp
-L Device:R R106
+L Device:R R100
 U 1 1 5F3A014C
 P 6800 5150
-F 0 "R106" H 6870 5196 50  0000 L CNN
+F 0 "R100" H 6870 5196 50  0000 L CNN
 F 1 "100k" H 6870 5105 50  0000 L CNN
 F 2 "Resistor_SMD:R_0402_1005Metric" V 6730 5150 50  0001 C CNN
@@
 	6800 4850 6800 5000
 $Comp
-L Device:R R110
+L Device:R R104
 U 1 1 5F3A0154
 P 7150 5150
-F 0 "R110" H 7220 5196 50  0000 L CNN
+F 0 "R104" H 7220 5196 50  0000 L CNN
 F 1 "100k" H 7220 5105 50  0000 L CNN
 F 2 "Resistor_SMD:R_0402_1005Metric" V 7080 5150 50  0001 C CNN

Commit message: relayout
Parts:
- renumbered C40 to C35, C41 to C36, C42 to C37, C43 to C38, J12 to J11, J13 to J12, J14 to J13, J15 to J14, R93 to R100, R94 to R101, R95 to R102, R96 to R103, R97 to R104, R98 to R105, R99 to R106, R100 to R107, R101 to R108, R102 to R109, R103 to R110, R104 to R111, U14 to U16, Y3 to Y1
Connections:
- net GND: now also J11.1 (Pin_1), J12.1 (Pin_1), J13.1 (Pin_1), J14.1 (Pin_1); no longer J11.4 (Pin_4), J12.4 (Pin_4), J13.4 (Pin_4), J14.4 (Pin_4)
- net RX0: now also R104.2; no longer R108.2
- net RX1: now also R105.2; no longer R109.2
- net RX2: now also R106.2; no longer R110.2
- net RX3: now also R107.2; no longer R111.2
- net TX0: now also J11.4 (Pin_4), R108.2; no longer J11.2 (Pin_2), R104.2
- net TX1: now also J12.4 (Pin_4), R109.2; no longer J12.2 (Pin_2), R105.2
- net TX2: now also J13.4 (Pin_4), R110.2; no longer J13.2 (Pin_2), R106.2
- net TX3: now also J14.4 (Pin_4), R111.2; no longer J14.2 (Pin_2), R107.2
- net VCC: now also J11.2 (Pin_2), J12.2 (Pin_2), J13.2 (Pin_2), J14.2 (Pin_2); no longer J11.1 (Pin_1), J12.1 (Pin_1), J13.1 (Pin_1), J14.1 (Pin_1)
Other:
- moved on the sheet: J11, J12, J13, J14

Commit message: modify planes
Parts:
- renumbered J11 to UART0, J12 to UART1, J13 to UART2, J14 to UART3
Changed lines of the file:
@@
 $Descr A4 11693 8268
 encoding utf-8
-Sheet 6 8
+Sheet 6 9
 Title ""
 Date ""
@@
 P 7900 3050
 AR Path="/5F37ABAA" Ref="J?"  Part="1"
-AR Path="/5F6EB2F1/5F37ABAA" Ref="J11"  Part="1"
-F 0 "J11" H 7928 3026 50  0000 L CNN
+AR Path="/5F6EB2F1/5F37ABAA" Ref="UART0"  Part="1"
+F 0 "UART0" H 7928 3026 50  0000 L CNN
 F 1 "Conn_01x04_Female" H 7928 2935 50  0000 L CNN
 F 2 "Connector_Molex:Molex_PicoBlade_53261-0471_1x04-1MP_P1.25mm_Horizontal" H 7900 3050 50  0001 C CNN
@@
 P 7900 3800
 AR Path="/5F37ABB1" Ref="J?"  Part="1"
-AR Path="/5F6EB2F1/5F37ABB1" Ref="J12"  Part="1"
-F 0 "J12" H 7928 3776 50  0000 L CNN
+AR Path="/5F6EB2F1/5F37ABB1" Ref="UART1"  Part="1"
+F 0 "UART1" H 7928 3776 50  0000 L CNN
 F 1 "Conn_01x04_Female" H 7928 3685 50  0000 L CNN
 F 2 "Connector_Molex:Molex_PicoBlade_53261-0471_1x04-1MP_P1.25mm_Horizontal" H 7900 3800 50  0001 C CNN
@@
 P 7900 4550
 AR Path="/5F37ABB8" Ref="J?"  Part="1"
-AR Path="/5F6EB2F1/5F37ABB8" Ref="J13"  Part="1"
-F 0 "J13" H 7928 4526 50  0000 L CNN
+AR Path="/5F6EB2F1/5F37ABB8" Ref="UART2"  Part="1"
+F 0 "UART2" H 7928 4526 50  0000 L CNN
 F 1 "Conn_01x04_Female" H 7928 4435 50  0000 L CNN
 F 2 "Connector_Molex:Molex_PicoBlade_53261-0471_1x04-1MP_P1.25mm_Horizontal" H 7900 4550 50  0001 C CNN
@@
 P 7900 5300
 AR Path="/5F37ABBF" Ref="J?"  Part="1"
-AR Path="/5F6EB2F1/5F37ABBF" Ref="J14"  Part="1"
-F 0 "J14" H 7928 5276 50  0000 L CNN
+AR Path="/5F6EB2F1/5F37ABBF" Ref="UART3"  Part="1"
+F 0 "UART3" H 7928 5276 50  0000 L CNN
 F 1 "Conn_01x04_Female" H 7928 5185 50  0000 L CNN
 F 2 "Connector_Molex:Molex_PicoBlade_53261-0471_1x04-1MP_P1.25mm_Horizontal" H 7900 5300 50  0001 C CNN

Commit message: added h bridge and magnetometers
Parts:
- R104, R105, R106, R107, R108, R109, R110, R111: Digikey Part Number 311-100KLRCT-ND -> YAG2307CT-ND
Changed lines of the file:
@@
 $Descr A4 11693 8268
 encoding utf-8
-Sheet 6 9
+Sheet 6 10
 Title ""
 Date ""
@@
 F 1 "100k" H 6870 2855 50  0000 L CNN
 F 2 "Resistor_SMD:R_0402_1005Metric" V 6730 2900 50  0001 C CNN
-F 3 "https://www.yageo.com/upload/media/product/productsearch/datasheet/rchip/PYu-RC_Group_51_RoHS_L_11.pdf" H 6800 2900 50  0001 C CNN
-F 4 "311-100KLRCT-ND" H 6800 2900 50  0001 C CNN "Digikey Part Number"
+F 3 "https://www.yageo.com/upload/media/product/productsearch/datasheet/rchip/PYu-RC_Group_51_RoHS_L_11.pdfhttps://www.yageo.com/upload/media/product/productsearch/datasheet/rchip/PYu-RT_1-to-0.01_RoHS_L_12.pdf" H 6800 2900 50  0001 C CNN
+F 4 "YAG2307CT-ND" H 6800 2900 50  0001 C CNN "Digikey Part Number"
 	1    6800 2900
 	1    0    0    -1
@@
 F 1 "100k" H 7220 2855 50  0000 L CNN
 F 2 "Resistor_SMD:R_0402_1005Metric" V 7080 2900 50  0001 C CNN
-F 3 "https://www.yageo.com/upload/media/product/productsearch/datasheet/rchip/PYu-RC_Group_51_RoHS_L_11.pdf" H 7150 2900 50  0001 C CNN
-F 4 "311-100KLRCT-ND" H 7150 2900 50  0001 C CNN "Digikey Part Number"
+F 3 "https://www.yageo.com/upload/media/product/productsearch/datasheet/rchip/PYu-RC_Group_51_RoHS_L_11.pdfhttps://www.yageo.com/upload/media/product/productsearch/datasheet/rchip/PYu-RT_1-to-0.01_RoHS_L_12.pdf" H 7150 2900 50  0001 C CNN
+F 4 "YAG2307CT-ND" H 7150 2900 50  0001 C CNN "Digikey Part Number"
 	1    7150 2900
 	1    0    0    -1
@@
 F 1 "100k" H 6870 3605 50  0000 L CNN
 F 2 "Resistor_SMD:R_0402_1005Metric" V 6730 3650 50  0001 C CNN
-F 3 "https://www.yageo.com/upload/media/product/productsearch/datasheet/rchip/PYu-RC_Group_51_RoHS_L_11.pdf" H 6800 3650 50  0001 C CNN
-F 4 "311-100KLRCT-ND" H 6800 3650 50  0001 C CNN "Digikey Part Number"
+F 3 "https://www.yageo.com/upload/media/product/productsearch/datasheet/rchip/PYu-RC_Group_51_RoHS_L_11.pdfhttps://www.yageo.com/upload/media/product/productsearch/datasheet/rchip/PYu-RT_1-to-0.01_RoHS_L_12.pdf" H 6800 3650 50  0001 C CNN
+F 4 "YAG2307CT-ND" H 6800 3650 50  0001 C CNN "Digikey Part Number"
 	1    6800 3650
 	1    0    0    -1
@@
 F 1 "100k" H 7220 3605 50  0000 L CNN
 F 2 "Resistor_SMD:R_0402_1005Metric" V 7080 3650 50  0001 C CNN
-F 3 "https://www.yageo.com/upload/media/product/productsearch/datasheet/rchip/PYu-RC_Group_51_RoHS_L_11.pdf" H 7150 3650 50  0001 C CNN
-F 4 "311-100KLRCT-ND" H 7150 3650 50  0001 C CNN "Digikey Part Number"
+F 3 "https://www.yageo.com/upload/media/product/productsearch/datasheet/rchip/PYu-RC_Group_51_RoHS_L_11.pdfhttps://www.yageo.com/upload/media/product/productsearch/datasheet/rchip/PYu-RT_1-to-0.01_RoHS_L_12.pdf" H 7150 3650 50  0001 C CNN
+F 4 "YAG2307CT-ND" H 7150 3650 50  0001 C CNN "Digikey Part Number"
 	1    7150 3650
 	1    0    0    -1
@@
 F 1 "100k" H 6870 4355 50  0000 L CNN
 F 2 "Resistor_SMD:R_0402_1005Metric" V 6730 4400 50  0001 C CNN
-F 3 "https://www.yageo.com/upload/media/product/productsearch/datasheet/rchip/PYu-RC_Group_51_RoHS_L_11.pdf" H 6800 4400 50  0001 C CNN
-F 4 "311-100KLRCT-ND" H 6800 4400 50  0001 C CNN "Digikey Part Number"
+F 3 "https://www.yageo.com/upload/media/product/productsearch/datasheet/rchip/PYu-RC_Group_51_RoHS_L_11.pdfhttps://www.yageo.com/upload/media/product/productsearch/datasheet/rchip/PYu-RT_1-to-0.01_RoHS_L_12.pdf" H 6800 4400 50  0001 C CNN
+F 4 "YAG2307CT-ND" H 6800 4400 50  0001 C CNN "Digikey Part Number"
 	1    6800 4400
 	1    0    0    -1
@@
 F 1 "100k" H 7220 4355 50  0000 L CNN
 F 2 "Resistor_SMD:R_0402_1005Metric" V 7080 4400 50  0001 C CNN
-F 3 "https://www.yageo.com/upload/media/product/productsearch/datasheet/rchip/PYu-RC_Group_51_RoHS_L_11.pdf" H 7150 4400 50  0001 C CNN
-F 4 "311-100KLRCT-ND" H 7150 4400 50  0001 C CNN "Digikey Part Number"
+F 3 "https://www.yageo.com/upload/media/product/productsearch/datasheet/rchip/PYu-RC_Group_51_RoHS_L_11.pdfhttps://www.yageo.com/upload/media/product/productsearch/datasheet/rchip/PYu-RT_1-to-0.01_RoHS_L_12.pdf" H 7150 4400 50  0001 C CNN
+F 4 "YAG2307CT-ND" H 7150 4400 50  0001 C CNN "Digikey Part Number"
 	1    7150 4400
 	1    0    0    -1
@@
 F 1 "100k" H 6870 5105 50  0000 L CNN
 F 2 "Resistor_SMD:R_0402_1005Metric" V 6730 5150 50  0001 C CNN
-F 3 "https://www.yageo.com/upload/media/product/productsearch/datasheet/rchip/PYu-RC_Group_51_RoHS_L_11.pdf" H 6800 5150 50  0001 C CNN
-F 4 "311-100KLRCT-ND" H 6800 5150 50  0001 C CNN "Digikey Part Number"
+F 3 "https://www.yageo.com/upload/media/product/productsearch/datasheet/rchip/PYu-RC_Group_51_RoHS_L_11.pdfhttps://www.yageo.com/upload/media/product/productsearch/datasheet/rchip/PYu-RT_1-to-0.01_RoHS_L_12.pdf" H 6800 5150 50  0001 C CNN
+F 4 "YAG2307CT-ND" H 6800 5150 50  0001 C CNN "Digikey Part Number"
 	1    6800 5150
 	1    0    0    -1
@@
 F 1 "100k" H 7220 5105 50  0000 L CNN
 F 2 "Resistor_SMD:R_0402_1005Metric" V 7080 5150 50  0001 C CNN
-F 3 "https://www.yageo.com/upload/media/product/productsearch/datasheet/rchip/PYu-RC_Group_51_RoHS_L_11.pdf" H 7150 5150 50  0001 C CNN
-F 4 "311-100KLRCT-ND" H 7150 5150 50  0001 C CNN "Digikey Part Number"
+F 3 "https://www.yageo.com/upload/media/product/productsearch/datasheet/rchip/PYu-RC_Group_51_RoHS_L_11.pdfhttps://www.yageo.com/upload/media/product/productsearch/datasheet/rchip/PYu-RT_1-to-0.01_RoHS_L_12.pdf" H 7150 5150 50  0001 C CNN
+F 4 "YAG2307CT-ND" H 7150 5150 50  0001 C CNN "Digikey Part Number"
 	1    7150 5150
 	1    0    0    -1
